File: Hardware/SCX3.sch (EAGLE design)
At the start: 175 parts, among them IC1 MAX604, IC10 ULN2074BN, IC2 LM339D, IC3 LM339D, IC4 LM339D, IC5 LM324N, IC6 LM324N, IC7 LM324N, IC8 MAX3221CAE, IC9 PIC32, K1 G6K-2P-Y, Q1 20MHz 18pF, Q4 BC848SMD, U1 AM10CW-2405S-NZ, U2 TEN3-2422WIN

Commit message: Release 1.1.0
Parts:
- removed Q4: BC848SMD, transistor-npn:BC848SMD
- removed R88: 4K7, rcl:R-EU_R0805
- removed R89: 1K, rcl:R-EU_R0805
- removed RS-232: (no value), ServoController:F09VP
- added C46: 27p, rcl:C-EUC0805
- added IC11: M95040, SCX3:M95040
- added Q2: 20MHz 18pF, crystal:CRYSTALSM49
- added R75, R76: 22K, rcl:R-EU_R0805
- added R78: 1K, rcl:R-EU_R0805
- added R80: 100, rcl:R-EU_R0805
- added R83: 4K7, rcl:R-EU_R0805
- added RS232: RJ-9, SCX3:RJ-9
- C11, C12, C13: value 10uF -> 100n
- C14: value 33n -> 100n
- C15, C17: value 10n -> 10uF
- C16: value 33n -> 10uF
- C18, C19, C28: value 33n -> 10n
- C2: value 1uF -> 220uF; device rcl:C-EUC0805 -> rcl:CPOL-EUE5-10.5
- C22, C25: value 10n -> 33n
- C29: value 100n -> 10n
- C3, C35: device rcl:C-EUC0805 -> rcl:CPOL-EUUD-4X5,8
- C30, C31, C32: value 100n -> 33n
- C33: device rcl:CPOL-EUUD-4X5,8 -> rcl:C-EUC0805
- C38, C41: value 27p -> 100n
- C4, C8: value 1nF/2KV -> 1uF
- C45: value 100n -> 27p
- C5: value 470uF -> 1nF/1KV
- C6: value 200uF -> 1nF/1KV; device rcl:CPOL-EUE5-10.5 -> rcl:C-EUC0805
- C7: value 470uF -> 10uF
- C9: value 10uF -> 1uF; device rcl:CPOL-EUUD-4X5,8 -> rcl:C-EUC0805
- IC10: value ULN2074BN -> PIC32MK1024MCF064; device uln-udn:ULN2074BN -> ServoController:PIC32MK1024MCF064
- IC2: value LM339D -> ULN2074BN; device linear:LM339D -> uln-udn:ULN2074BN
- IC5: value LM324N -> LM339D; device ServoController:LM324N -> linear:LM339D
- IC8: value MAX3221CAE -> LM324N; device ServoController:MAX3221CAE -> ServoController:LM324N
- IC9: value PIC32 -> MAX3221CAE; device ServoController:PIC32MK1024MCF0649X9MM -> ServoController:MAX3221CAE
- LED3: value LED -12V -> LED 5V
- LED4: value LED 5V -> LED 3V3
- LED5: value LED 3V3 -> LED -12V
- OK1: value TLP2662F -> LTV844; device ServoController:TLP2662F -> ServoController:LTV844
- OK4: value LTV844 -> TLP2662F; device ServoController:LTV844 -> ServoController:TLP2662F
- Q1: value 20MHz 18pF -> BC848SMD; device crystal:CRYSTALSM49 -> transistor-npn:BC848SMD
- R12, R13: value 470 -> 4K7
- R16, R18, R23, R24: value 4K7 -> 470
- R2, R3: value 470 -> 1K; POWER 0.19W -> (none)
- R27: value 330 -> 4K7
- R28, R84: value 1K -> 4K7
- R29, R33, R37: value 47K -> 4K7
- R30: value 22K -> 1K
- R31: value 22K -> 470
- R32: value 10K -> 4K7
- R34, R35, R36: value 22K -> 4K7
- R39, R52, R58, R65: value 10K -> 22K
- R4: value 130 -> 330; POWER 52mW -> (none)
- R41, R42, R50, R54, R55: value 47K -> 22K
- R44, R47, R48, R49: value 22K -> 10K
- R46: value 47K -> 10K
- R5: POWER 10mW -> (none)
- R56, R60, R64: value 22K -> 47K
- R6, R7: value 4K7 -> 1K
- R68, R69, R70: value 100 -> 47K; POWER 10mW -> (none)
- R71: value 10K -> 47K
- R72: value 1K -> 47K
- R73: value 4K7 -> 47K
- R74: value 1K -> 22K
- R77: value 4K7 -> 10K
- R79: value 1K -> 100
- R8, R9: value 470 -> 1K
- R81: value 4K7 -> 100
- U1: value AM10CW-2405S-NZ -> AM6T-2412D-NZ; device ServoController:AM10CW-2405S-NZ -> SCX3:AM6T-2412D-NZ
- U2: value TEN3-2422WIN -> AM10CW-2405S-NZ; device ServoController:TEN3-2422WIN -> ServoController:AM10CW-2405S-NZ
Connections:
- removed net 24V_F: C1.+, C2.1, C4.1, C6.+, D1.C, F1.2, INTERFACE.15, K11.+, L1.1, LED1.A, U2.+VIN
- removed net 2V5: R27.1, R28.2, SJ1.1, SJ2.1, SJ3.1, SJ4.1, SJ5.1, SJ6.1, SJ7.1, SJ8.1, SJ9.1
- new net !HOLD: IC11.!HOLD, R84.2
- new net !MSS: IC10.TRCLK/RPC6/PWM6H/RC6, IC11.!CS, R83.2
- new net !MWP: IC10.SOSCI/RPC13/RC13, IC11.!WP, R82.2
- new net MSCK: IC10.TRD0/RPC7/PWM12H/PWM6L/RC7, IC11.SCK
- new net MSDI: IC10.SOSCO/RPB8/RB8, IC11.SO
- new net MSDO: IC10.TMS/OA5IN-/AN27/CVD27/C5IN1-/RPB9/RB9, IC11.SI
- new net N$12: F1.1, POWER-1.KL
- new net REF: R30.1, R31.2, SJ10.1, SJ2.1, SJ3.1, SJ4.1, SJ5.1, SJ6.1, SJ7.1, SJ8.1, SJ9.1
- net !MCLR: now also IC10.!MCLR, R78.2; no longer IC9.!MCLR, R72.2
- net +12V: now also C5.2, C8.1, IC8P.V+, OUTPUT.5, U1.+VOUT; no longer C4.2, C5.1, IC5P.V+, U2.+VOUT
- net -12V: now also C6.1, C9.2, IC8P.V-, LED5.C, OUTPUT.4, U1.-VOUT; no longer C7.2, C8.1, IC5P.V-, LED3.C, U2.-VOUT
- net 24V: now also C1.+, C2.+, C4.1, C5.1, F1.2, INTERFACE.15, L1.1, LED1.A, U1.+VIN; no longer F1.1, POWER-1.KL
- net 24VGND: now also C2.-, C4.2, C6.2, U1.-VIN, U2.-IN; no longer C2.2, C6.-, C8.2, U1.-IN, U2.-VIN
- net 3V3: now also C35.+, C41.2, C42.2, C43.2, C44.1, C7.1, IC10.AVDD, IC10.VDD@1, IC10.VDD@2, IC10.VDD@3, IC10.VDD@4, IC10.VUSB3V3, IC11.VCC, IC5P.V+, IC9G$1.!FORCEOFF, IC9P.VCC, LED4.A, OK4P.VCC, R12.2, R13.2, R27.2, R28.2, R29.2, R32.2, R33.2, R34.2, R35.2, R36.2, R37.2, R83.1, R84.1; no longer C10.1, C33.+, C35.2, C36.2, C37.1, IC2P.V+, IC8G$1.!FORCEOFF, IC8P.VCC, IC9.AVDD, IC9.VDD@1, IC9.VDD@2, IC9.VDD@3, IC9.VDD@4, IC9.VUSB3V3, LED5.A, OK1P.VCC, R14.2, R16.2, R18.2, R23.2, R24.2, R6.2, R7.2, R71.2, R73.2, R82.2, R88.2
- net 5V: now also C10.1, C15.2, C16.2, C17.2, C3.+, D1.C, K11.+, LED3.A, R30.2, U2.+OUT; no longer C11.2, C12.2, C13.2, C3.1, C9.+, LED4.A, R27.2, U1.+OUT
- net CH1_A+: now also IC3A.+IN; no longer IC2A.+IN
- net CH1_A-: now also IC3A.-IN, SJ2.2; no longer IC2A.-IN, SJ1.2
- net CH1_B+: now also IC3B.+IN; no longer IC2B.+IN
- net CH1_B-: now also IC3B.-IN, SJ3.2; no longer IC2B.-IN, SJ4.2
- net CH1_CMD: now also IC6D.-IN, IC6D.OUT; no longer IC5D.-IN, IC5D.OUT
- net CH1_DIR: now also IC10.OA3OUT/AN6/CVD6/C3IN4-/C4IN1+/C4IN4-/RPC0/RC0, OK2B.VO, R19.1; no longer IC9.OA3OUT/AN6/CVD6/C3IN4-/C4IN1+/C4IN4-/RPC0/RC0, OK1B.VO, R10.1
- net CH1_DIR_H: now also R16.1; no longer R12.1
- net CH1_DIR_L: now also OK2B.C; no longer OK1B.C
- net CH1_H: now also IC10.RPB14/PWM1H/VBUSON1/PMPD6/RB14, R38.1; no longer IC9.RPB14/PWM1H/VBUSON1/PMPD6/RB14, R31.1
- net CH1_I+: now also IC3C.+IN; no longer IC2C.+IN
- net CH1_I-: now also IC3C.-IN, SJ4.2; no longer IC2C.-IN, SJ7.2
- net CH1_L: now also IC10.RPB15/PWM7H/PWM1L/PMPD7/RB15, R39.1; no longer IC9.RPB15/PWM7H/PWM1L/PMPD7/RB15, R38.1
- net CH1_QE_A: now also IC10.AN15/CVD15/RPE15/FLT8/PMPA0/PSPA0/RE15, IC3A.OUT, R27.1; no longer IC2A.OUT, IC9.TDI/DAC3/AN26/CVD26/RPA8/PMPA9/RA8, R18.1
- net CH1_QE_B: now also IC10.OA5IN+/DAC1/AN24/CVD24/C5IN1+/C5IN3-/RPA4/T1CK/T1G/RA4, IC3B.OUT, R28.1; no longer IC2B.OUT, IC9.AN15/CVD15/RPE15/FLT8/PMPA0/PSPA0/RE15, R21.1
- net CH1_QE_I: now also IC10.TDI/DAC3/AN26/CVD26/RPA8/PMPA9/RA8, IC3C.OUT, R29.1; no longer IC2C.OUT, IC9.OA5IN+/DAC1/AN24/CVD24/C5IN1+/C5IN3-/RPA4/T1CK/T1G/RA4, R24.1
- net CH1_STEP: now also IC10.PGED1/OA1IN-/AN5/CTCMP/C1IN1-/RTCC/RPB3/RB3, OK2A.VO, R21.1; no longer IC9.PGED1/OA1IN-/AN5/CTCMP/C1IN1-/RTCC/RPB3/RB3, OK1A.VO, R6.1
- net CH1_STEP_H: now also R15.1; no longer R8.1
- net CH1_STEP_L: now also OK2A.C; no longer OK1A.C
- net CH2_A+: now also IC4A.+IN; no longer IC3A.+IN
- net CH2_A-: now also IC4A.-IN, SJ5.2; no longer IC3A.-IN, SJ2.2
- net CH2_B+: now also IC4B.+IN; no longer IC3B.+IN
- net CH2_B-: now also IC4B.-IN, SJ6.2; no longer IC3B.-IN, SJ5.2
- net CH2_CMD: now also IC7D.-IN, IC7D.OUT; no longer IC6D.-IN, IC6D.OUT
- net CH2_DIR: now also IC10.FLT15/RPB4/PMPA8/RB4, OK4B.VO, R25.1; no longer IC9.FLT15/RPB4/PMPA8/RB4, OK2B.VO, R11.1
- net CH2_DIR_H: now also R24.1; no longer R13.1
- net CH2_DIR_L: now also OK4B.C; no longer OK2B.C
- net CH2_H: now also IC10.TDO/PWM4H/PMPD4/RA10, R40.1; no longer IC9.TDO/PWM4H/PMPD4/RA10, R44.1
- net CH2_I+: now also IC4C.+IN; no longer IC3C.+IN
- net CH2_I-: now also IC4C.-IN, SJ7.2; no longer IC3C.-IN, SJ8.2
- net CH2_L: now also IC10.TCK/RPA7/PWM10H/PWM4L/PMPD5/RA7, R41.1; no longer IC9.TCK/RPA7/PWM10H/PWM4L/PMPD5/RA7, R51.1
- net CH2_QE_A: now also IC10.OA3IN+/AN8/CVD8/C3IN1+/C3IN3-/RPC2/FLT3/PMPA13/RC2, IC4A.OUT, R32.1; no longer IC3A.OUT, IC9.OA3IN+/AN8/CVD8/C3IN1+/C3IN3-/RPC2/FLT3/PMPA13/RC2, R19.1
- net CH2_QE_B: now also IC10.OA3IN-/AN7/CVD7/C3IN1-/C4IN1-/RPC1/PMPA7/RC1, IC4B.OUT, R33.1; no longer IC3B.OUT, IC9.OA3IN-/AN7/CVD7/C3IN1-/C4IN1-/RPC1/PMPA7/RC1, R22.1
- net CH2_QE_I: now also IC10.PGEC3/OA1OUT/VREF+/AN3/C1IN4-/C4IN2-/RPB1/CTED1/PMPA6/RB1, IC4C.OUT, R34.1; no longer IC3C.OUT, IC9.PGEC3/OA1OUT/VREF+/AN3/C1IN4-/C4IN2-/RPB1/CTED1/PMPA6/RB1, R25.1
- net CH2_STEP: now also IC10.AN14/CVD14/RPE14/FLT7/PMPA1/PSPA1/RE14, OK4A.VO, R26.1; no longer IC9.AN14/CVD14/RPE14/FLT7/PMPA1/PSPA1/RE14, OK2A.VO, R7.1
- net CH2_STEP_H: now also R23.1; no longer R9.1
- net CH2_STEP_L: now also OK4A.C; no longer OK2A.C
- net CH3_A+: now also IC5A.+IN; no longer IC4A.+IN
- net CH3_A-: now also IC5A.-IN, SJ8.2; no longer IC4A.-IN, SJ3.2
- net CH3_B+: now also IC5B.+IN; no longer IC4B.+IN
- net CH3_B-: now also IC5B.-IN, SJ9.2; no longer IC4B.-IN, SJ6.2
- net CH3_CMD: now also IC8D.-IN, IC8D.OUT; no longer IC7D.-IN, IC7D.OUT
- net CH3_DIR: now also IC10.AN11/CVD11/C1IN2-/FLT4/PMPA12/RC11, R20.1; no longer IC9.AN11/CVD11/C1IN2-/FLT4/PMPA12/RC11, R16.1
- net CH3_DIR_H: now also R18.1; no longer R17.1
- net CH3_H: now also IC10.RPB12/PWM2H/PMPD2/RB12, R42.1; no longer IC9.RPB12/PWM2H/PMPD2/RB12, R57.1
- net CH3_I+: now also IC5C.+IN; no longer IC4C.+IN
- net CH3_I-: now also IC5C.-IN, SJ10.2; no longer IC4C.-IN, SJ9.2
- net CH3_L: now also IC10.RPB13/PWM8H/PWM2L/CTPLS/PMPD3/RB13, R43.1; no longer IC9.RPB13/PWM8H/PWM2L/CTPLS/PMPD3/RB13, R64.1
- net CH3_QE_A: now also IC10.OA2OUT/ANO/C2IN4-/C4IN3-/RPA0/RA0, IC5A.OUT, R35.1; no longer IC4A.OUT, IC9.OA2OUT/ANO/C2IN4-/C4IN3-/RPA0/RA0, R20.1
- net CH3_QE_B: now also IC10.OA2IN+/AN1/C2IN1+/RPA1/RA1, IC5B.OUT, R36.1; no longer IC4B.OUT, IC9.OA2IN+/AN1/C2IN1+/RPA1/RA1, R23.1
- net CH3_QE_I: now also IC10.PGEC1/OA1IN+/AN4/C1IN1+/C1IN3-/C2IN3-/RPB2/RB2, IC5C.OUT, R37.1; no longer IC4C.OUT, IC9.PGEC1/OA1IN+/AN4/C1IN1+/C1IN3-/C2IN3-/RPB2/RB2, R26.1
- net CH3_STEP: now also IC10.PGED3/VREF-/OA2IN-/AN2/C2IN1-/RPB0/CTED2/RB0, R22.1; no longer IC9.PGED3/VREF-/OA2IN-/AN2/C2IN1-/RPB0/CTED2/RB0, R14.1
- net CH3_STEP_H: now also R17.1; no longer R15.1
- net DI1: now also IC10.AN19/CVD19/RPG6/PMPA5/RG6, OK1A.C, R10.1; no longer IC9.AN19/CVD19/RPG6/PMPA5/RG6, OK4A.C, R73.1
- net DI1_CON: now also R6.1; no longer R74.1
- net DI2: now also IC10.AN18/CVD18/RPG7/PMPA4/RG7, OK1B.C, R11.1; no longer IC9.AN18/CVD18/RPG7/PMPA4/RG7, OK4B.C, R77.1
- net DI2_CON: now also R7.1; no longer R79.1
- net DI3: now also IC10.AN17/CVD17/RPG8/PMPA3/RG8, OK1C.C, R12.1; no longer IC9.AN17/CVD17/RPG8/PMPA3/RG8, OK4C.C, R82.1
- net DI3_CON: now also R8.1; no longer R84.1
- net DI4: now also IC10.AN16/CVD16/RPG9/PMPA2/RG9, OK1D.C, R13.1; no longer IC9.AN16/CVD16/RPG9/PMPA2/RG9, OK4D.C, R88.1
- net DI4_CON: now also R9.1; no longer R89.1
- net DI_COM_CON: now also C11.2, C12.2, C13.2, C14.2, OK1A.AC2, OK1B.AC2, OK1C.AC2, OK1D.AC2; no longer C42.2, C43.2, C44.2, C45.2, OK4A.AC2, OK4B.AC2, OK4C.AC2, OK4D.AC2
- net DO1: now also IC10.TRD1/RPC8/PWM5H/PMPWR/PSPWR/RC8, IC2.I4; no longer IC10.I4, IC9.TRD1/RPC8/PWM5H/PMPWR/PSPWR/RC8
- net DO1H_CON: now also Q1.C; no longer Q4.C
- net DO1_CON: now also IC2.C4; no longer IC10.C4
- net DO2: now also IC10.TRD2/RPD5/PWM12H/PMPRD/PSPRD/RD5, IC2.I3; no longer IC10.I3, IC9.TRD2/RPD5/PWM12H/PMPRD/PSPRD/RD5
- net DO2_CON: now also IC2.C3; no longer IC10.C3
- net DO3: now also IC10.AN10/CVD10/RPA12/RA12, IC2.I1; no longer IC10.I1, IC9.AN10/CVD10/RPA12/RA12
- net DO3_CON: now also IC2.C1; no longer IC10.C1
- net DO4: now also IC10.AN9/CVD9/RPA11/USBOEN1/RA11, IC2.I2; no longer IC10.I2, IC9.AN9/CVD9/RPA11/USBOEN1/RA11
- net DO4_CON: now also IC2.C2; no longer IC10.C2
- net DO_COM_CON: now also IC2.E1, IC2.E2, IC2.E3, IC2.E4, SJ1.2; no longer IC10.E1, IC10.E2, IC10.E3, IC10.E4, SJ10.2
- net GND: now also C15.1, C16.1, C17.1, C21.1, C22.2, C23.1, C24.2, C25.1, C3.-, C30.2, C35.-, C36.2, C42.1, C43.1, C44.2, C45.1, C46.1, C7.2, C8.2, C9.1, IC10.AVSS, IC10.VSS@1, IC10.VSS@2, IC10.VSS@3, IC10.VSS@4, IC11.VSS, IC2.SUB1, IC2.SUB2, IC2.SUB3, IC2.SUB4, IC5P.GND, IC9G$1.!EN, IC9G$1.FORCEON, IC9P.GND, OK1A.E, OK1B.E, OK1C.E, OK1D.E, OK4P.GND, Q1.E, R31.1, R56.2, R60.2, R63.1, R64.2, R68.1, R70.1, R72.1, R82.1, RS232.1, RS232.4, SJ1.1, U1.COM, U2.-OUT; no longer C11.1, C12.1, C13.1, C14.1, C16.2, C18.2, C19.1, C21.2, C23.2, C24.1, C28.2, C3.2, C33.-, C34.1, C35.1, C36.1, C5.2, C7.1, C9.-, IC10.SUB1, IC10.SUB2, IC10.SUB3, IC10.SUB4, IC2P.GND, IC8G$1.!EN, IC8G$1.FORCEON, IC8P.GND, IC9.AVSS, IC9.VSS@1, IC9.VSS@2, IC9.VSS@3, IC9.VSS@4, OK1P.GND, OK4A.E, OK4B.E, OK4C.E, OK4D.E, Q4.E, R28.1, R29.2, R33.1, R41.1, R42.2, R46.1, R54.1, R55.2, RS-232.5, RS-232.G1, RS-232.G2, SJ10.1, U1.-OUT, U2.COM
- net LED_ERROR: now also IC10.RPB10/PWM3H/PMPD0/RB10, R81.1; no longer IC9.RPB10/PWM3H/PMPD0/RB10, R70.1
- net LED_READY: now also IC10.RPF0/PWM11H/RF0, R79.1; no longer IC9.RPF0/PWM11H/RF0, R68.1
- net LED_STATE: now also IC10.RPF1/PWM11L/RF1, R80.1; no longer IC9.RPF1/PWM11L/RF1, R69.1
- net N$1: now also IC6B.-IN, R51.1, R59.2; no longer IC5B.-IN, R40.1, R41.2
- net N$10: now also IC6C.-IN, R58.1, R69.1; no longer IC5C.-IN, R36.1, R37.1
- net N$11: now also C27.2, IC6B.OUT, R51.2, R58.2; no longer C17.2, IC5B.OUT, R36.2, R40.2
- net N$13: now also C22.1, IC6B.+IN, R45.2; no longer C18.1, IC5B.+IN, R39.2
- net N$14: now also C27.1, R39.2, R45.1; no longer C17.1, R38.2, R39.1
- net N$15: now also IC6C.+IN, R57.1, R68.2; no longer IC5C.+IN, R33.2, R34.1
- net N$16: now also OK4B.A, R24.2; no longer OK2B.A, R13.2
- net N$17: now also OK4A.A, R23.2; no longer OK2A.A, R9.2
- net N$18: now also R18.2; no longer R17.2
- net N$19: now also R17.2; no longer R15.2
- net N$2: now also IC6A.-IN, R50.2, R56.1; no longer IC5A.-IN, R29.1, R30.2
- net N$20: now also IC7B.-IN, R63.2; no longer IC6B.-IN, R54.2
- net N$21: now also IC7A.-IN, R52.2, R60.1; no longer IC6A.-IN, R42.1, R43.2
- net N$22: now also C19.1, IC7A.OUT, R52.1, R61.2; no longer C20.1, IC6A.OUT, R43.1, R47.2
- net N$23: now also C23.2, IC7A.+IN, R46.2; no longer C19.2, IC6A.+IN, R45.2
- net N$24: now also C19.2, R40.2, R46.1; no longer C20.2, R44.2, R45.1
- net N$25: now also C31.1, IC7D.+IN, R75.2; no longer C21.1, IC6D.+IN, R48.2
- net N$26: now also IC7C.OUT, R71.2, R75.1; no longer IC6C.OUT, R48.1, R50.2
- net N$27: now also IC7C.-IN, R62.1, R71.1; no longer IC6C.-IN, R49.1, R50.1
- net N$28: now also C28.2, IC7B.OUT, R62.2; no longer C22.2, IC6B.OUT, R49.2
- net N$29: now also C24.1, IC7B.+IN, R47.2; no longer C23.1, IC6B.+IN, R52.2
- net N$30: now also C28.1, R41.2, R47.1; no longer C22.1, R51.2, R52.1
- net N$31: now also IC7C.+IN, R61.1, R70.2; no longer IC6C.+IN, R46.2, R47.1
- net N$32: now also IC8B.-IN, R55.1; no longer IC7B.-IN, R66.1
- net N$33: now also IC8A.-IN, R54.2, R64.1; no longer IC7A.-IN, R55.1, R56.2
- net N$34: now also C20.1, IC8A.OUT, R54.1, R65.2; no longer C25.1, IC7A.OUT, R56.1, R60.2
- net N$35: now also C25.2, IC8A.+IN, R48.2; no longer C24.2, IC7A.+IN, R58.2
- net N$36: now also C20.2, R42.2, R48.1; no longer C25.2, R57.2, R58.1
- net N$37: now also C32.1, IC8D.+IN, R76.2; no longer C26.1, IC7D.+IN, R61.2
- net N$38: now also IC8C.OUT, R73.2, R76.1; no longer IC7C.OUT, R61.1, R63.2
- net N$39: now also IC8C.-IN, R66.1, R73.1; no longer IC7C.-IN, R62.1, R63.1
- net N$4: now also U2.+IN; no longer U1.+IN
- net N$40: now also C29.2, IC8B.OUT, R55.2; no longer C27.2, IC7B.OUT, R62.2
- net N$41: now also C26.1, IC8B.+IN, R49.2; no longer C28.1, IC7B.+IN, R65.2
- net N$42: now also C29.1, R43.2, R49.1; no longer C27.1, R64.2, R65.1
- net N$43: now also IC8C.+IN, R65.1, R72.2; no longer IC7C.+IN, R59.2, R60.1
- net N$45: now also R79.2; no longer R68.2
- net N$47: now also R80.2; no longer R69.2
- net N$48: now also R81.2; no longer R70.2
- net N$5: now also C18.1, IC6A.OUT, R50.1, R57.2; no longer C15.1, IC5A.OUT, R30.1, R34.2
- net N$50: now also C34.2, IC9G$1.C1-; no longer C30.2, IC8G$1.C1-
- net N$51: now also C34.1, IC9G$1.C1+; no longer C30.1, IC8G$1.C1+
- net N$52: now also C33.2, IC9G$1.C2-; no longer C29.2, IC8G$1.C2-
- net N$53: now also C33.1, IC9G$1.C2+; no longer C29.1, IC8G$1.C2+
- net N$54: now also C36.1, IC9G$1.V+; no longer C31.1, IC8G$1.V+
- net N$55: now also C37.1, IC9G$1.V-; no longer C32.1, IC8G$1.V-
- net N$56: now also C12.1, OK1B.AC1, R7.2; no longer C43.1, OK4B.AC1, R79.2
- net N$6: now also C21.2, IC6A.+IN, R44.2; no longer C14.2, IC5A.+IN, R32.2
- net N$65: now also LED3.C; no longer LED4.C
- net N$67: now also C38.2, R77.1, R78.1; no longer C34.2, R71.1, R72.1
- net N$69: now also Q1.B, R14.2; no longer Q4.B, R81.2
- net N$7: now also C18.2, R38.2, R44.1; no longer C15.2, R31.2, R32.1
- net N$70: now also C13.1, OK1C.AC1, R8.2; no longer C44.1, OK4C.AC1, R84.2
- net N$71: now also C14.1, OK1D.AC1, R9.2; no longer C45.1, OK4D.AC1, R89.2
- net N$72: now also C11.1, OK1A.AC1, R6.2; no longer C42.1, OK4A.AC1, R74.2
- net N$73: now also OK2B.A, R16.2; no longer OK1B.A, R12.2
- net N$74: now also OK2A.A, R15.2; no longer OK1A.A, R8.2
- net N$75: now also LED4.C; no longer LED5.C
- net N$76: now also LED5.A; no longer LED3.A
- net N$8: now also C30.1, IC6D.+IN, R74.2; no longer C16.1, IC5D.+IN, R35.2
- net N$9: now also IC6C.OUT, R69.2, R74.1; no longer IC5C.OUT, R35.1, R37.2
- net OSC1I: now also C45.2, IC10.OSCI/CLKI/AN49/CVD49/RPC12/RC12, Q2.2; no longer C38.2, IC9.OSCI/CLKI/AN49/CVD49/RPC12/RC12, Q1.2
- net OSC1O: now also C46.2, IC10.OSCO/CLKO/RPC15/RC15, Q2.1; no longer C41.2, IC9.OSCO/CLKO/RPC15/RC15, Q1.1
- net PGEC: now also IC10.PGEC2/RPB6/SCK2/PMPA15/RB6; no longer IC9.PGEC2/RPB6/SCK2/PMPA15/RB6
- net PGED: now also IC10.PGED2/RPB5/USBID1/RB5; no longer IC9.PGED2/RPB5/USBID1/RB5
- net RO1: now also IC10.RPB11/PWM9H/PWM3L/PMPD1/RB11, R14.1; no longer IC9.RPB11/PWM9H/PWM3L/PMPD1/RB11, R81.1
- net RS232_RX: now also IC9G$1.R1IN, RS232.2; no longer IC8G$1.R1IN, RS-232.2
- net RS232_TX: now also IC9G$1.T1OUT, RS232.3; no longer IC8G$1.T1OUT, RS-232.3
- net UART_RX: now also IC10.RPC9/PWM11H/PWM5L/RC9, IC9G$1.R1OUT; no longer IC8G$1.R1OUT, IC9.RPC9/PWM11H/PWM5L/RC9
- net UART_TX: now also IC10.TRD3/RPD6/PWM12L/RD6, IC9G$1.T1IN; no longer IC8G$1.T1IN, IC9.TRD3/RPD6/PWM12L/RD6
Other:
- note removed: "10-15mA"
- note removed: "10mA"
- note removed: "2-2,5V"
- note removed: "20mA"

Commit message: Release 1.2.0
Parts:
- removed C37, C38, C39: 100n, rcl:C-EUC0805
- removed IC9: MAX3221CAE, ServoController:MAX3221CAE
- removed LED4: LED 3V3, led:LEDSML1206
- removed R1: 2K2, rcl:R-EU_R1206
- removed R4: 330, rcl:R-EU_R0805
- removed R7: 1K, rcl:R-EU_R0805
- removed RS232: RJ-9, SCX3:RJ-9
- added C47, C50: 100n, rcl:C-EUC0805
- added C55: 100n, rcl:CPOL-EUUD-4X5,8
- added D2, D3: 1N4148, diode:1N4148SMD-0805
- added D4: ESD5Z3.3, diode:ZENER-DIODESOD523
- added F2: 0.63A, fuse:TR5
- added IC13: MAX3089, MyLib:MAX3089
- added L2: 4,7uH, MyLib:DJNR6028--S
- added LED14: LED READY, led:LEDSML1206
- added LED16: LED ERROR, led:LEDSML1206
- added LED19: TX, led:LEDSML0603
- added LED20: RX, led:LEDSML0603
- added Q3, Q4: BC848, transistor-npn:BC848SMD
- added R85, R88, R89: 100, rcl:R-EU_R0805
- added R86, R87, R90: 4K7, rcl:R-EU_R0805
- added R91: 10K, rcl:R-EU_R0805
- added R92: 1K, rcl:R-EU_R0805
- added R95, R96: 100, rcl:R-EU_R0603
- added R97: 10K, rcl:R-EU_R0603
- added RS485-IN, RS485-OUT: RJ-45-SH_RJSS-88-A22-E1V, MyLib:RJ-45-SH_RJSS-88-A22-E1V
- added S1: DIP-6_TDA06H0_SB1, MyLib:DIP-6_TDA06H0_SB1
- added USB: USB, MyLib:DIP-USB-B-TYPE-FMAL(4+2P-2.5-90D)
- C1: value 330uF -> 1nF/1KV; device rcl:CPOL-EUE5-10.5 -> rcl:C-EUC1206
- C10: value 10uF -> 1uF
- C11, C14: value 100n -> 10uF
- C12: value 100n -> 1nF/1KV; device rcl:C-EUC0805 -> rcl:C-EUC1206
- C13: value 100n -> 10uF; device rcl:C-EUC0805 -> rcl:CPOL-EUUD-4X5,8
- C15, C16, C17: value 10uF -> 100n
- C18: value 10n -> 100n
- C19, C20: value 10n -> 10uF
- C2: value 220uF -> 1uF; device rcl:CPOL-EUE5-10.5 -> rcl:C-EUC0805
- C21: value 33n -> 10uF
- C23, C25, C30: value 33n -> 10n
- C27, C29: value 10n -> 33n
- C3: value 10uF -> 1000uF; device rcl:CPOL-EUUD-4X5,8 -> rcl:CPOL-EUE5-10.5
- C33: value 100n -> 10n
- C34, C36: value 100n -> 33n
- C35: value 100n -> 10n; device rcl:CPOL-EUUD-4X5,8 -> rcl:C-EUC0805
- C43, C44: value 100n -> 27p
- C45, C46: value 27p -> 100n
- C5: value 1nF/1KV -> 10uF
- C6: value 1nF/1KV -> 1uF
- C7: value 10uF -> 1nF/1KV; device rcl:C-EUC0805 -> rcl:C-EUC1206
- C8: value 1uF -> 1nF/1KV; device rcl:C-EUC0805 -> rcl:C-EUC1206
- C9: value 1uF -> 330uF; device rcl:C-EUC0805 -> rcl:CPOL-EUE5-10.5
- D1: value 1N4148SMD-0805 -> 1N4148
- ENCODER1, ENCODER2, ENCODER3, OUTPUT: device ServoController:F09VP -> con-subd:F09VP
- F1: value 3A -> 0.63A; device fuse:SH22,5 -> fuse:TR5
- IC1: device ServoController:MAX604 -> MyLib:MAX604
- IC10: value PIC32MK1024MCF064 -> M95040; device ServoController:PIC32MK1024MCF064 -> MyLib:M95040
- IC11: value M95040 -> PIC32MK1024MCF064; device SCX3:M95040 -> MyLib:PIC32MK1024MCF064
- IC6, IC7, IC8: device ServoController:LM324N -> MyLib:LM324N
- ICSP: device ServoController:JP5E -> MyLib:JP5E
- K1: device ServoController:G6K-2P-Y -> MyLib:G6K-2P-Y
- L1: device ServoController:DJNR6028--S -> MyLib:DJNR6028--S
- LED1: value LED 24V -> (none); device led:LEDSML1206 -> led:DUOLED-RG-C
- LED2: value LED +12V -> (none); device led:LEDSML1206 -> led:DUOLED-RG-C
- LED3: value LED 5V -> LED +12V
- LED6: value LED READY -> LED 5V
- LED8: value LED ERROR -> LED 3V3
- OK1: device ServoController:LTV844 -> MyLib:LTV844
- OK2, OK3, OK4: device ServoController:TLP2662F -> MyLib:TLP2662F
- R11, R13: value 4K7 -> 470; device rcl:R-EU_R0805 -> rcl:R-EU_R1206; WATTAGE (none) -> 500mW
- R15, R17: value 470 -> 1K
- R16, R18, R23, R24, R31: value 470 -> 4K7
- R19, R22: value 4K7 -> 1K
- R2, R9: value 1K -> 470; device rcl:R-EU_R0805 -> rcl:R-EU_R1206; WATTAGE (none) -> 500mW
- R25, R26, R29, R32, R34: value 4K7 -> 470
- R30: value 1K -> 470
- R38, R39, R40, R41, R42, R43: value 22K -> 4K7
- R44: value 10K -> 1K
- R45: value 10K -> 470
- R46: value 10K -> 47K
- R47, R48, R77: value 10K -> 22K
- R5: value 100 -> 1K
- R50, R54, R58, R76: value 22K -> 47K
- R56, R69: value 47K -> 10K
- R6: value 1K -> 330
- R60, R64, R68, R70, R73: value 47K -> 22K
- R62, R75: value 22K -> 10K
- R78: value 1K -> 22K
- R79, R81: value 100 -> 22K
- R8: value 1K -> 100
- R80: value 100 -> 47K
- R82: value 4K7 -> 10K
- R83: value 4K7 -> 22K
- R84: value 4K7 -> 47K
- U1: value AM6T-2412D-NZ -> AM6C-2412D-NZ; device SCX3:AM6T-2412D-NZ -> MyLib:AM6C-2412D-NZ
- U2: device ServoController:AM10CW-2405S-NZ -> MyLib:AM10CW-2405S-NZ
- renumbered C40 to C48, C41 to C49, LED7 to LED15
Connections:
- net DO1H_CON renamed N$12
- removed net 24V: C1.+, C2.+, C4.1, C5.1, F1.2, INTERFACE.15, L1.1, LED1.A, U1.+VIN
- removed net N$12 (its old number): F1.1, POWER-1.KL
- removed net N$3: LED1.C, R1.1
- removed net N$50: C34.2, IC9G$1.C1-
- removed net N$51: C34.1, IC9G$1.C1+
- removed net N$52: C33.2, IC9G$1.C2-
- removed net N$53: C33.1, IC9G$1.C2+
- removed net N$54: C36.1, IC9G$1.V+
- removed net N$55: C37.1, IC9G$1.V-
- removed net RS232_RX: IC9G$1.R1IN, RS232.2
- removed net RS232_TX: IC9G$1.T1OUT, RS232.3
- new net 24V_1: C3.+, C4.1, D2.A, F1.2, L1.1
- new net 24V_2: C10.1, C9.+, D3.A, F2.2, L2.1
- new net 24V_SUPPLY: F1.1, F2.1, POWER-1.KL, R2.1, R9.1
- new net H/!F: IC13G$1.H/!F, S1.12
- new net N$46: C1.1, L1.2, U1.+VIN
- new net N$49: LED1.AR, Q3.C, R9.2
- new net N$57: Q3.B, R10.2
- new net N$59: LED1.AG, R11.1
- new net N$60: D2.C, R10.1, R11.2
- new net N$61: LED2.AR, Q4.C, R2.2
- new net N$66: Q4.B, R12.2
- new net N$68: LED2.AG, R13.1
- new net N$77: D3.C, R12.1, R13.2
- new net N$82: LED19.A, R95.2
- new net N$83: LED20.A, R96.2
- new net N$85: R97.1, S1.9
- new net RS485_A: IC13G$1.A, RS485-IN.5, RS485-OUT.5
- new net RS485_B: IC13G$1.B, RS485-IN.8, RS485-OUT.8
- new net RS485_Y: IC13G$1.Y, RS485-IN.1, RS485-OUT.1
- new net RS485_Z: IC13G$1.Z, RS485-IN.4, RS485-OUT.4
- new net RXP: IC13G$1.RXP, S1.10
- new net SLR: IC13G$1.SLR, R97.2, S1.8
- new net TXP: IC13G$1.TXP, S1.11
- new net UART_!CTS: IC11.OA5OUT/AN25/CVD25/C5IN4-/RPB7/SCK1/INT0/RB7, IC13G$1.!RE, IC13G$1.DE
- new net UART_!RTR: IC11.DAC2/AN48/CVD48/RPC10/PMPA14/PSPCS/RC10
- new net USB_D+: IC11.D+, USB.1
- new net USB_D-: IC11.D-, USB.2
- new net VBUS: IC11.VBUS, USB.3
- net !HOLD: now also IC10.!HOLD, R87.2; no longer IC11.!HOLD, R84.2
- net !MCLR: now also IC11.!MCLR, R92.2; no longer IC10.!MCLR, R78.2
- net !MSS: now also IC10.!CS, IC11.TRCLK/RPC6/PWM6H/RC6, R86.2; no longer IC10.TRCLK/RPC6/PWM6H/RC6, IC11.!CS, R83.2
- net !MWP: now also IC10.!WP, IC11.SOSCI/RPC13/RC13, R90.2; no longer IC10.SOSCI/RPC13/RC13, IC11.!WP, R82.2
- net +12V: now also C1.2, C2.1, C5.1, LED3.A; no longer C5.2, C8.1, LED2.A
- net -12V: now also C5.2, C6.2, C7.1; no longer C6.1, C9.2
- net 24VGND: now also C10.2, C12.2, C3.-, C7.2, C9.-, LED1.C, LED2.C, Q3.E, Q4.E, U2.-VIN; no longer C1.-, C2.-, C6.2, R1.2, U2.-IN
- net 3V3: now also C14.1, C46.2, C47.2, C50.1, C55.+, D4.C, IC10.VCC, IC11.AVDD, IC11.VDD@1, IC11.VDD@2, IC11.VDD@3, IC11.VDD@4, IC11.VUSB3V3, IC13P.VCC, LED8.A, R14.2, R16.2, R18.2, R23.2, R24.2, R31.2, R38.2, R39.2, R40.2, R41.2, R42.2, R43.2, R86.1, R87.1, R91.2, R95.1, R96.1, S1.1, S1.2, S1.3, S1.4; no longer C35.+, C39.2, C43.2, C44.1, C7.1, IC10.AVDD, IC10.VDD@1, IC10.VDD@2, IC10.VDD@3, IC10.VDD@4, IC10.VUSB3V3, IC11.VCC, IC9G$1.!FORCEOFF, IC9P.VCC, LED4.A, R10.2, R11.2, R12.2, R13.2, R19.2, R20.2, R22.2, R25.2, R26.2, R29.2, R32.2, R34.2, R77.2, R83.1, R84.1
- net 5V: now also C11.1, C13.+, C19.2, C20.2, C21.2, C8.2, LED6.A, R44.2, U2.+VOUT; no longer C10.1, C15.2, C16.2, C17.2, C3.+, LED3.A, R30.2, U2.+OUT
- net CH1_A+: now also IC3B.+IN; no longer IC3A.+IN
- net CH1_A-: now also IC3B.-IN; no longer IC3A.-IN
- net CH1_B+: now also IC3A.+IN; no longer IC3B.+IN
- net CH1_B-: now also IC3A.-IN, SJ5.2; no longer IC3B.-IN, SJ3.2
- net CH1_DIR: now also IC11.OA3OUT/AN6/CVD6/C3IN4-/C4IN1+/C4IN4-/RPC0/RC0, R27.1; no longer IC10.OA3OUT/AN6/CVD6/C3IN4-/C4IN1+/C4IN4-/RPC0/RC0, R19.1
- net CH1_DIR_H: now also R29.1; no longer R16.1
- net CH1_H: now also IC11.RPB14/PWM1H/VBUSON1/PMPD6/RB14, R48.1; no longer IC10.RPB14/PWM1H/VBUSON1/PMPD6/RB14, R38.1
- net CH1_I-: now also SJ8.2; no longer SJ4.2
- net CH1_L: now also IC11.RPB15/PWM7H/PWM1L/PMPD7/RB15, R55.1; no longer IC10.RPB15/PWM7H/PWM1L/PMPD7/RB15, R39.1
- net CH1_QE_A: now also IC11.AN15/CVD15/RPE15/FLT8/PMPA0/PSPA0/RE15, IC3B.OUT, R38.1; no longer IC10.AN15/CVD15/RPE15/FLT8/PMPA0/PSPA0/RE15, IC3A.OUT, R27.1
- net CH1_QE_B: now also IC11.OA5IN+/DAC1/AN24/CVD24/C5IN1+/C5IN3-/RPA4/T1CK/T1G/RA4, IC3A.OUT, R35.1; no longer IC10.OA5IN+/DAC1/AN24/CVD24/C5IN1+/C5IN3-/RPA4/T1CK/T1G/RA4, IC3B.OUT, R28.1
- net CH1_QE_I: now also IC11.TDI/DAC3/AN26/CVD26/RPA8/PMPA9/RA8, R41.1; no longer IC10.TDI/DAC3/AN26/CVD26/RPA8/PMPA9/RA8, R29.1
- net CH1_STEP: now also IC11.PGED1/OA1IN-/AN5/CTCMP/C1IN1-/RTCC/RPB3/RB3, R23.1; no longer IC10.PGED1/OA1IN-/AN5/CTCMP/C1IN1-/RTCC/RPB3/RB3, R21.1
- net CH1_STEP_H: now also R25.1; no longer R15.1
- net CH2_A-: now also SJ3.2; no longer SJ5.2
- net CH2_DIR: now also IC11.FLT15/RPB4/PMPA8/RB4, OK3B.VO, R28.1; no longer IC10.FLT15/RPB4/PMPA8/RB4, OK4B.VO, R25.1
- net CH2_DIR_H: now also R30.1; no longer R24.1
- net CH2_DIR_L: now also OK3B.C; no longer OK4B.C
- net CH2_H: now also IC11.TDO/PWM4H/PMPD4/RA10, R61.1; no longer IC10.TDO/PWM4H/PMPD4/RA10, R40.1
- net CH2_I-: now also SJ9.2; no longer SJ7.2
- net CH2_L: now also IC11.TCK/RPA7/PWM10H/PWM4L/PMPD5/RA7, R68.1; no longer IC10.TCK/RPA7/PWM10H/PWM4L/PMPD5/RA7, R41.1
- net CH2_QE_A: now also IC11.OA3IN+/AN8/CVD8/C3IN1+/C3IN3-/RPC2/FLT3/PMPA13/RC2, R36.1; no longer IC10.OA3IN+/AN8/CVD8/C3IN1+/C3IN3-/RPC2/FLT3/PMPA13/RC2, R32.1
- net CH2_QE_B: now also IC11.OA3IN-/AN7/CVD7/C3IN1-/C4IN1-/RPC1/PMPA7/RC1, R39.1; no longer IC10.OA3IN-/AN7/CVD7/C3IN1-/C4IN1-/RPC1/PMPA7/RC1, R33.1
- net CH2_QE_I: now also IC11.PGEC3/OA1OUT/VREF+/AN3/C1IN4-/C4IN2-/RPB1/CTED1/PMPA6/RB1, R42.1; no longer IC10.PGEC3/OA1OUT/VREF+/AN3/C1IN4-/C4IN2-/RPB1/CTED1/PMPA6/RB1, R34.1
- net CH2_STEP: now also IC11.AN14/CVD14/RPE14/FLT7/PMPA1/PSPA1/RE14, OK3A.VO, R24.1; no longer IC10.AN14/CVD14/RPE14/FLT7/PMPA1/PSPA1/RE14, OK4A.VO, R26.1
- net CH2_STEP_H: now also R26.1; no longer R23.1
- net CH2_STEP_L: now also OK3A.C; no longer OK4A.C
- net CH3_A-: now also SJ4.2; no longer SJ8.2
- net CH3_B-: now also SJ7.2; no longer SJ9.2
- net CH3_DIR: now also IC11.AN11/CVD11/C1IN2-/FLT4/PMPA12/RC11, OK4B.VO, R33.1; no longer IC10.AN11/CVD11/C1IN2-/FLT4/PMPA12/RC11, OK3B.VO, R20.1
- net CH3_DIR_H: now also R34.1; no longer R18.1
- net CH3_DIR_L: now also OK4B.C; no longer OK3B.C
- net CH3_H: now also IC11.RPB12/PWM2H/PMPD2/RB12, R74.1; no longer IC10.RPB12/PWM2H/PMPD2/RB12, R42.1
- net CH3_L: now also IC11.RPB13/PWM8H/PWM2L/CTPLS/PMPD3/RB13, R81.1; no longer IC10.RPB13/PWM8H/PWM2L/CTPLS/PMPD3/RB13, R43.1
- net CH3_QE_A: now also IC11.OA2OUT/ANO/C2IN4-/C4IN3-/RPA0/RA0, R37.1; no longer IC10.OA2OUT/ANO/C2IN4-/C4IN3-/RPA0/RA0, R35.1
- net CH3_QE_B: now also IC11.OA2IN+/AN1/C2IN1+/RPA1/RA1, R40.1; no longer IC10.OA2IN+/AN1/C2IN1+/RPA1/RA1, R36.1
- net CH3_QE_I: now also IC11.PGEC1/OA1IN+/AN4/C1IN1+/C1IN3-/C2IN3-/RPB2/RB2, R43.1; no longer IC10.PGEC1/OA1IN+/AN4/C1IN1+/C1IN3-/C2IN3-/RPB2/RB2, R37.1
- net CH3_STEP: now also IC11.PGED3/VREF-/OA2IN-/AN2/C2IN1-/RPB0/CTED2/RB0, OK4A.VO, R31.1; no longer IC10.PGED3/VREF-/OA2IN-/AN2/C2IN1-/RPB0/CTED2/RB0, OK3A.VO, R22.1
- net CH3_STEP_H: now also R32.1; no longer R17.1
- net CH3_STEP_L: now also OK4A.C; no longer OK3A.C
- net DI1: now also IC11.AN19/CVD19/RPG6/PMPA5/RG6, R14.1; no longer IC10.AN19/CVD19/RPG6/PMPA5/RG6, R10.1
- net DI1_CON: now also R15.1; no longer R6.1
- net DI2: now also IC11.AN18/CVD18/RPG7/PMPA4/RG7, R16.1; no longer IC10.AN18/CVD18/RPG7/PMPA4/RG7, R11.1
- net DI2_CON: now also R17.1; no longer R7.1
- net DI3: now also IC11.AN17/CVD17/RPG8/PMPA3/RG8, R18.1; no longer IC10.AN17/CVD17/RPG8/PMPA3/RG8, R12.1
- net DI3_CON: now also R19.1; no longer R8.1
- net DI4: now also IC11.AN16/CVD16/RPG9/PMPA2/RG9, R21.1; no longer IC10.AN16/CVD16/RPG9/PMPA2/RG9, R13.1
- net DI4_CON: now also R22.1; no longer R9.1
- net DI_COM_CON: now also C15.2, C16.2, C17.2, C18.2; no longer C11.2, C12.2, C13.2, C14.2
- net DO1: now also IC11.TRD1/RPC8/PWM5H/PMPWR/PSPWR/RC8; no longer IC10.TRD1/RPC8/PWM5H/PMPWR/PSPWR/RC8
- net DO2: now also IC11.TRD2/RPD5/PWM12H/PMPRD/PSPRD/RD5; no longer IC10.TRD2/RPD5/PWM12H/PMPRD/PSPRD/RD5
- net DO3: now also IC11.AN10/CVD10/RPA12/RA12; no longer IC10.AN10/CVD10/RPA12/RA12
- net DO4: now also IC11.AN9/CVD9/RPA11/USBOEN1/RA11; no longer IC10.AN9/CVD9/RPA11/USBOEN1/RA11
- net GND: now also C11.2, C12.1, C13.-, C14.2, C19.1, C2.2, C20.1, C22.1, C27.1, C29.2, C32.1, C34.2, C44.1, C47.1, C50.2, C55.-, C6.1, D4.A, IC10.VSS, IC11.AVSS, IC11.VSS@1, IC11.VSS@2, IC11.VSS@3, IC11.VSS@4, IC13P.GND, LED14.C, LED16.C, R45.1, R46.2, R50.1, R58.1, R59.2, R6.2, R71.1, R72.2, R76.1, R8.2, R84.1, R90.1, RS485-IN.3, RS485-IN.SH, RS485-OUT.3, RS485-OUT.SH, S1.5, U2.-VOUT, USB.4, USB.5; no longer C10.2, C15.1, C16.1, C17.1, C22.2, C23.1, C25.1, C3.-, C30.2, C32.2, C35.-, C37.2, C38.1, C39.1, C44.2, C7.2, C8.2, C9.1, IC10.AVSS, IC10.VSS@1, IC10.VSS@2, IC10.VSS@3, IC10.VSS@4, IC11.VSS, IC9G$1.!EN, IC9G$1.FORCEON, IC9P.GND, LED6.C, LED8.C, R2.2, R31.1, R4.2, R56.2, R59.1, R60.2, R64.2, R67.1, R68.1, R70.1, R72.1, R82.1, RS232.1, RS232.4, U2.-OUT
- net LED_ERROR: now also IC11.RPB10/PWM3H/PMPD0/RB10, R89.1; no longer IC10.RPB10/PWM3H/PMPD0/RB10, R81.1
- net LED_READY: now also IC11.RPF0/PWM11H/RF0, R85.1; no longer IC10.RPF0/PWM11H/RF0, R79.1
- net LED_STATE: now also IC11.RPF1/PWM11L/RF1, R88.1; no longer IC10.RPF1/PWM11L/RF1, R80.1
- net MSCK: now also IC10.SCK, IC11.TRD0/RPC7/PWM12H/PWM6L/RC7; no longer IC10.TRD0/RPC7/PWM12H/PWM6L/RC7, IC11.SCK
- net MSDI: now also IC10.SO, IC11.SOSCO/RPB8/RB8; no longer IC10.SOSCO/RPB8/RB8, IC11.SO
- net MSDO: now also IC10.SI, IC11.TMS/OA5IN-/AN27/CVD27/C5IN1-/RPB9/RB9; no longer IC10.TMS/OA5IN-/AN27/CVD27/C5IN1-/RPB9/RB9, IC11.SI
- net N$1: now also R57.1, R58.2; no longer R51.1, R59.2
- net N$10: now also R53.1, R54.1; no longer R58.1, R69.1
- net N$11: now also C25.2, R53.2, R57.2; no longer C27.2, R51.2, R58.2
- net N$13: now also C26.1, R56.2; no longer C22.1, R45.2
- net N$14: now also C25.1, R55.2, R56.1; no longer C27.1, R39.2, R45.1
- net N$15: now also R50.2, R51.1; no longer R57.1, R68.2
- net N$16: now also OK3B.A, R30.2; no longer OK4B.A, R24.2
- net N$17: now also OK3A.A, R26.2; no longer OK4A.A, R23.2
- net N$18: now also OK4B.A, R34.2; no longer OK3B.A, R18.2
- net N$19: now also OK4A.A, R32.2; no longer OK3A.A, R17.2
- net N$2: now also R46.1, R47.2; no longer R50.2, R56.1
- net N$20: now also R70.1, R71.2; no longer R53.1, R63.2
- net N$21: now also R59.1, R60.2; no longer R52.2, R60.1
- net N$22: now also C28.1, R60.1, R64.2; no longer C19.1, R52.1, R61.2
- net N$23: now also C27.2, R62.2; no longer C23.2, R46.2
- net N$24: now also C28.2, R61.2, R62.1; no longer C19.2, R40.2, R46.1
- net N$25: now also C29.1, R65.2; no longer C31.1, R75.2
- net N$26: now also R65.1, R67.2; no longer R71.2, R75.1
- net N$27: now also R66.1, R67.1; no longer R62.1, R71.1
- net N$28: now also C30.2, R66.2, R70.2; no longer C28.2, R53.2, R62.2
- net N$29: now also C31.1, R69.2; no longer C24.1, R47.2
- net N$30: now also C30.1, R68.2, R69.1; no longer C28.1, R41.2, R47.1
- net N$31: now also R63.2, R64.1; no longer R61.1, R70.2
- net N$32: now also R83.1, R84.2; no longer R55.1, R67.2
- net N$33: now also R72.1, R73.2; no longer R54.2, R64.1
- net N$34: now also C33.1, R73.1, R77.2; no longer C20.1, R54.1, R65.2
- net N$35: now also C32.2, R75.2; no longer C25.2, R48.2
- net N$36: now also C33.2, R74.2, R75.1; no longer C20.2, R42.2, R48.1
- net N$37: now also C34.1, R78.2; no longer C32.1, R76.2
- net N$38: now also R78.1, R80.2; no longer R73.2, R76.1
- net N$39: now also R79.1, R80.1; no longer R66.1, R73.1
- net N$4: now also C8.1, L2.2, U2.+VIN; no longer L1.2, U2.+IN
- net N$40: now also C35.2, R79.2, R83.2; no longer C29.2, R55.2, R66.2
- net N$41: now also C36.1, R82.2; no longer C26.1, R49.2
- net N$42: now also C35.1, R81.2, R82.1; no longer C29.1, R43.2, R49.1
- net N$43: now also R76.2, R77.1; no longer R65.1, R72.2
- net N$45: now also LED14.A, R85.2; no longer LED6.A, R79.2
- net N$47: now also R88.2; no longer R80.2
- net N$48: now also LED16.A, R89.2; no longer LED8.A, R81.2
- net N$5: now also C23.1, R47.1, R51.2; no longer C18.1, R50.1, R57.2
- net N$56: now also C16.1, R17.2; no longer C12.1, R7.2
- net N$58: now also LED3.C, R3.1; no longer LED2.C, R2.1
- net N$6: now also C22.2, R49.2; no longer C21.2, R44.2
- net N$65: now also LED6.C, R6.1; no longer LED3.C, R4.1
- net N$67: now also C45.2, R91.1, R92.1; no longer C38.2, R77.1, R78.1
- net N$69: now also R20.2; no longer R14.2
- net N$7: now also C23.2, R48.2, R49.1; no longer C18.2, R38.2, R44.1
- net N$70: now also C17.1, R19.2; no longer C13.1, R8.2
- net N$71: now also C18.1, R22.2; no longer C14.1, R9.2
- net N$72: now also C15.1, R15.2; no longer C11.1, R6.2
- net N$73: now also R29.2; no longer R16.2
- net N$74: now also R25.2; no longer R15.2
- net N$75: now also LED8.C, R8.1; no longer LED4.C, R5.1
- net N$76: now also R5.1; no longer R3.1
- net N$8: now also C24.1, R52.2; no longer C30.1, R74.2
- net N$9: now also R52.1, R54.2; no longer R69.2, R74.1
- net OSC1I: now also C43.2, IC11.OSCI/CLKI/AN49/CVD49/RPC12/RC12; no longer C45.2, IC10.OSCI/CLKI/AN49/CVD49/RPC12/RC12
- net OSC1O: now also C44.2, IC11.OSCO/CLKO/RPC15/RC15; no longer C46.2, IC10.OSCO/CLKO/RPC15/RC15
- net PGEC: now also IC11.PGEC2/RPB6/SCK2/PMPA15/RB6; no longer IC10.PGEC2/RPB6/SCK2/PMPA15/RB6
- net PGED: now also IC11.PGED2/RPB5/USBID1/RB5; no longer IC10.PGED2/RPB5/USBID1/RB5
- net REF: now also R44.1, R45.2; no longer R30.1, R31.2
- net RO1: now also IC11.RPB11/PWM9H/PWM3L/PMPD1/RB11, R20.1; no longer IC10.RPB11/PWM9H/PWM3L/PMPD1/RB11, R14.1
- net UART_RX: now also IC11.RPC9/PWM11H/PWM5L/RC9, IC13G$1.RO, LED20.C; no longer IC10.RPC9/PWM11H/PWM5L/RC9, IC9G$1.R1OUT
- net UART_TX: now also IC11.TRD3/RPD6/PWM12L/RD6, IC13G$1.DI, LED19.C; no longer IC10.TRD3/RPD6/PWM12L/RD6, IC9G$1.T1IN
