File: Hardware/SCX3.brd (EAGLE design)
At the start: 157 x 72 mm, 175 parts, among them IC1 MAX604, IC10 ULN2074BN, IC2 LM339D, IC3 LM339D, IC4 LM339D, IC5 LM324N, IC6 LM324N, IC7 LM324N, IC8 MAX3221CAE, IC9 PIC32, K1 G6K-2P-Y, Q1 20MHz 18pF, Q4 BC848SMD, U1 AM10CW-2405S-NZ, U2 TEN3-2422WIN

Commit message: Release 1.1.0
Parts:
- removed Q4: BC848SMD, transistor-npn:SOT23
- removed R88: 4K7, rcl:R0805
- removed R89: 1K, rcl:R0805
- removed RS-232: (no value), ServoController:F09VP
- added C46: 27p, rcl:C0805
- added IC11: M95040, SCX3:SO8
- added Q2: 20MHz 18pF, crystal:SM49
- added R75, R76: 22K, rcl:R0805
- added R78: 1K, rcl:R0805
- added R80: 100, rcl:R0805
- added R83: 4K7, rcl:R0805
- added RS232: RJ-9, SCX3:RJ-9
- C11, C12, C13: value 10uF -> 100n
- C14: value 33n -> 100n
- C15, C17: value 10n -> 10uF
- C16: value 33n -> 10uF
- C18, C19, C28: value 33n -> 10n
- C2: value 1uF -> 220uF; device rcl:C0805 -> rcl:E5-10,5
- C22, C25: value 10n -> 33n
- C29: value 100n -> 10n
- C3, C35: device rcl:C0805 -> rcl:UD-4X5,8_NICHICON
- C30, C31, C32: value 100n -> 33n
- C33: device rcl:UD-4X5,8_NICHICON -> rcl:C0805
- C38, C41: value 27p -> 100n
- C4, C8: value 1nF/2KV -> 1uF
- C45: value 100n -> 27p
- C5: value 470uF -> 1nF/1KV
- C6: value 200uF -> 1nF/1KV; device rcl:E5-10,5 -> rcl:C0805
- C7: value 470uF -> 10uF
- C9: value 10uF -> 1uF; device rcl:UD-4X5,8_NICHICON -> rcl:C0805
- IC10: value ULN2074BN -> PIC32MK1024MCF064; device uln-udn:DIL16 -> ServoController:QFN64-9X9
- IC2: value LM339D -> ULN2074BN; device linear:SO14 -> uln-udn:DIL16
- IC5: value LM324N -> LM339D; device ServoController:DIL14 -> linear:SO14
- IC8: value MAX3221CAE -> LM324N; device ServoController:SSOP16 -> ServoController:DIL14
- IC9: value PIC32 -> MAX3221CAE; device ServoController:QFN64-9X9 -> ServoController:SSOP16
- LED3: value LED -12V -> LED 5V
- LED4: value LED 5V -> LED 3V3
- LED5: value LED 3V3 -> LED -12V
- OK1: value TLP2662F -> LTV844; device ServoController:DIL08 -> ServoController:DIL16
- OK4: value LTV844 -> TLP2662F; device ServoController:DIL16 -> ServoController:DIL08
- Q1: value 20MHz 18pF -> BC848SMD; device crystal:SM49 -> transistor-npn:SOT23
- R12, R13: value 470 -> 4K7
- R16, R18, R23, R24: value 4K7 -> 470
- R2, R3, R8, R9: value 470 -> 1K
- R27: value 330 -> 4K7
- R28, R84: value 1K -> 4K7
- R29, R33, R37: value 47K -> 4K7
- R30: value 22K -> 1K
- R31: value 22K -> 470
- R32: value 10K -> 4K7
- R34, R35, R36: value 22K -> 4K7
- R39, R52, R58, R65: value 10K -> 22K
- R4: value 130 -> 330
- R41, R42, R50, R54, R55: value 47K -> 22K
- R44, R47, R48, R49: value 22K -> 10K
- R46: value 47K -> 10K
- R56, R60, R64: value 22K -> 47K
- R6, R7: value 4K7 -> 1K
- R68, R69, R70: value 100 -> 47K
- R71: value 10K -> 47K
- R72: value 1K -> 47K
- R73: value 4K7 -> 47K
- R74: value 1K -> 22K
- R77: value 4K7 -> 10K
- R79: value 1K -> 100
- R81: value 4K7 -> 100
- U1: value AM10CW-2405S-NZ -> AM6T-2412D-NZ; device ServoController:AM10CW-NZ -> SCX3:AM6T
- U2: value TEN3-2422WIN -> AM10CW-2405S-NZ; device ServoController:TEN3-WIN -> ServoController:AM10CW-NZ
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Connections:
- removed net 24V_F: C1.+, C2.1, C4.1, C6.+, D1.2, F1.2, INTERFACE.15, K1.1, L1.A, LED1.A, U2.22, U2.23
- removed net 2V5: R27.1, R28.2, SJ1.1, SJ2.1, SJ3.1, SJ4.1, SJ5.1, SJ6.1, SJ7.1, SJ8.1, SJ9.1
- new net !HOLD: IC11.7, R84.2
- new net !MSS: IC10.50, IC11.1, R83.2
- new net !MWP: IC10.47, IC11.3, R82.2
- new net MSCK: IC10.51, IC11.6
- new net MSDI: IC10.48, IC11.2
- new net MSDO: IC10.49, IC11.5
- new net N$12: F1.1, POWER.1
- new net REF: R30.1, R31.2, SJ10.1, SJ2.1, SJ3.1, SJ4.1, SJ5.1, SJ6.1, SJ7.1, SJ8.1, SJ9.1
- net !MCLR: now also IC10.7, R78.2; no longer IC9.7, R72.2
- net +12V: now also C5.2, C8.1, IC8.4, OUTPUT.5, U1.14; no longer C4.2, C5.1, IC5.4, U2.14
- net -12V: now also C6.1, C9.2, IC8.11, LED5.C, OUTPUT.4, U1.11; no longer C7.2, C8.1, IC5.11, LED3.C, U2.11
- net 24V: now also C1.+, C2.+, C4.1, C5.1, F1.2, INTERFACE.15, L1.A, LED1.A, U1.22, U1.23; no longer F1.1, POWER.1
- net 24VGND: now also C2.-, C4.2, C6.2, U1.3; no longer C2.2, C6.-, C8.2, U2.3
- net 3V3: now also C35.+, C41.2, C42.2, C43.2, C44.1, C7.1, IC10.10, IC10.19, IC10.26, IC10.35, IC10.38, IC10.57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; no longer C10.1, C33.+, C35.2, C36.2, C37.1, IC2.3, IC8.15, IC8.16, IC9.10, IC9.19, IC9.26, IC9.35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
- net 5V: now also C10.1, C15.2, C16.2, C17.2, C3.+, D1.2, K1.1, LED3.A, R30.2, U2.4; no longer C11.2, C12.2, C13.2, C3.1, C9.+, LED4.A, R27.2, U1.4
- net CH1_A+: now also IC3.5; no longer IC2.5
- net CH1_A-: now also IC3.4, SJ2.2; no longer IC2.4, SJ1.2
- net CH1_B+: now also IC3.7; no longer IC2.7
- net CH1_B-: now also IC3.6, SJ3.2; no longer IC2.6, SJ4.2
- net CH1_CMD: now also IC6.13, IC6.14; no longer IC5.13, IC5.14
- net CH1_DIR: now also IC10.21, OK2.6, R19.1; no longer IC9.21, OK1.6, R10.1
- net CH1_DIR_H: now also R16.1; no longer R12.1
- net CH1_DIR_L: now also OK2.3; no longer OK1.3
- net CH1_H: now also IC10.2, R38.1; no longer IC9.2, R31.1
- net CH1_I+: now also IC3.9; no longer IC2.9
- net CH1_I-: now also IC3.8, SJ4.2; no longer IC2.8, SJ7.2
- net CH1_L: now also IC10.3, R39.1; no longer IC9.3, R38.1
- net CH1_QE_A: now also IC10.30, IC3.2, R27.1; no longer IC2.2, IC9.31, R18.1
- net CH1_QE_B: now also IC10.33, IC3.1, R28.1; no longer IC2.1, IC9.30, R21.1
- net CH1_QE_I: now also IC10.31, IC3.14, R29.1; no longer IC2.14, IC9.33, R24.1
- net CH1_STEP: now also IC10.18, OK2.7, R21.1; no longer IC9.18, OK1.7, R6.1
- net CH1_STEP_H: now also R15.1; no longer R8.1
- net CH1_STEP_L: now also OK2.2; no longer OK1.2
- net CH2_A+: now also IC4.5; no longer IC3.5
- net CH2_A-: now also IC4.4, SJ5.2; no longer IC3.4, SJ2.2
- net CH2_B+: now also IC4.7; no longer IC3.7
- net CH2_B-: now also IC4.6, SJ6.2; no longer IC3.6, SJ5.2
- net CH2_CMD: now also IC7.13, IC7.14; no longer IC6.13, IC6.14
- net CH2_DIR: now also IC10.32, OK4.6, R25.1; no longer IC9.32, OK2.6, R11.1
- net CH2_DIR_H: now also R24.1; no longer R13.1
- net CH2_DIR_L: now also OK4.3; no longer OK2.3
- net CH2_H: now also IC10.64, R40.1; no longer IC9.64, R44.1
- net CH2_I+: now also IC4.9; no longer IC3.9
- net CH2_I-: now also IC4.8, SJ7.2; no longer IC3.8, SJ8.2
- net CH2_L: now also IC10.1, R41.1; no longer IC9.1, R51.1
- net CH2_QE_A: now also IC10.23, IC4.2, R32.1; no longer IC3.2, IC9.23, R19.1
- net CH2_QE_B: now also IC10.22, IC4.1, R33.1; no longer IC3.1, IC9.22, R22.1
- net CH2_QE_I: now also IC10.16, IC4.14, R34.1; no longer IC3.14, IC9.16, R25.1
- net CH2_STEP: now also IC10.29, OK4.7, R26.1; no longer IC9.29, OK2.7, R7.1
- net CH2_STEP_H: now also R23.1; no longer R9.1
- net CH2_STEP_L: now also OK4.2; no longer OK2.2
- net CH3_A+: now also IC5.5; no longer IC4.5
- net CH3_A-: now also IC5.4, SJ8.2; no longer IC4.4, SJ3.2
- net CH3_B+: now also IC5.7; no longer IC4.7
- net CH3_B-: now also IC5.6, SJ9.2; no longer IC4.6, SJ6.2
- net CH3_CMD: now also IC8.13, IC8.14; no longer IC7.13, IC7.14
- net CH3_DIR: now also IC10.24, R20.1; no longer IC9.24, R16.1
- net CH3_DIR_H: now also R18.1; no longer R17.1
- net CH3_H: now also IC10.62, R42.1; no longer IC9.62, R57.1
- net CH3_I+: now also IC5.9; no longer IC4.9
- net CH3_I-: now also IC5.8, SJ10.2; no longer IC4.8, SJ9.2
- net CH3_L: now also IC10.63, R43.1; no longer IC9.63, R64.1
- net CH3_QE_A: now also IC10.13, IC5.2, R35.1; no longer IC4.2, IC9.13, R20.1
- net CH3_QE_B: now also IC10.14, IC5.1, R36.1; no longer IC4.1, IC9.14, R23.1
- net CH3_QE_I: now also IC10.17, IC5.14, R37.1; no longer IC4.14, IC9.17, R26.1
- net CH3_STEP: now also IC10.15, R22.1; no longer IC9.15, R14.1
- net CH3_STEP_H: now also R17.1; no longer R15.1
- net DI1: now also IC10.4, OK1.16, R10.1; no longer IC9.4, OK4.16, R73.1
- net DI1_CON: now also R6.1; no longer R74.1
- net DI2: now also IC10.5, OK1.14, R11.1; no longer IC9.5, OK4.14, R77.1
- net DI2_CON: now also R7.1; no longer R79.1
- net DI3: now also IC10.6, OK1.12, R12.1; no longer IC9.6, OK4.12, R82.1
- net DI3_CON: now also R8.1; no longer R84.1
- net DI4: now also IC10.8, OK1.10, R13.1; no longer IC9.8, OK4.10, R88.1
- net DI4_CON: now also R9.1; no longer R89.1
- net DI_COM_CON: now also C11.2, C12.2, C13.2, C14.2, OK1.2, OK1.4, OK1.6, OK1.8; no longer C42.2, C43.2, C44.2, C45.2, OK4.2, OK4.4, OK4.6, OK4.8
- net DO1: now also IC10.52, IC2.14; no longer IC10.14, IC9.52
- net DO1H_CON: now also Q1.3; no longer Q4.3
- net DO1_CON: now also IC2.16; no longer IC10.16
- net DO2: now also IC10.53, IC2.11; no longer IC10.11, IC9.53
- net DO2_CON: now also IC2.9; no longer IC10.9
- net DO3: now also IC10.11, IC2.3; no longer IC10.3, IC9.11
- net DO3_CON: now also IC2.1; no longer IC10.1
- net DO4: now also IC10.12, IC2.6; no longer IC10.6, IC9.12
- net DO4_CON: now also IC2.8; no longer IC10.8
- net DO_COM_CON: now also IC2.10, IC2.15, IC2.2, IC2.7, SJ1.2; no longer IC10.10, IC10.15, IC10.2, IC10.7, SJ10.2
- net GND: now also C15.1, C16.1, C17.1, C21.1, C22.2, C23.1, C24.2, C25.1, C3.-, C30.2, C35.-, C36.2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; no longer C11.1, C12.1, C13.1, C14.1, C16.2, C18.2, C19.1, C21.2, C23.2, C24.1, C28.2, C3.2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
- net LED_ERROR: now also IC10.60, R81.1; no longer IC9.60, R70.1
- net LED_READY: now also IC10.58, R79.1; no longer IC9.58, R68.1
- net LED_STATE: now also IC10.59, R80.1; no longer IC9.59, R69.1
- net N$1: now also IC6.6, R51.1, R59.2; no longer IC5.6, R40.1, R41.2
- net N$10: now also IC6.9, R58.1, R69.1; no longer IC5.9, R36.1, R37.1
- net N$11: now also C27.2, IC6.7, R51.2, R58.2; no longer C17.2, IC5.7, R36.2, R40.2
- net N$13: now also C22.1, IC6.5, R45.2; no longer C18.1, IC5.5, R39.2
- net N$14: now also C27.1, R39.2, R45.1; no longer C17.1, R38.2, R39.1
- net N$15: now also IC6.10, R57.1, R68.2; no longer IC5.10, R33.2, R34.1
- net N$16: now also OK4.4, R24.2; no longer OK2.4, R13.2
- net N$17: now also OK4.1, R23.2; no longer OK2.1, R9.2
- net N$18: now also R18.2; no longer R17.2
- net N$19: now also R17.2; no longer R15.2
- net N$2: now also IC6.2, R50.2, R56.1; no longer IC5.2, R29.1, R30.2
- net N$20: now also IC7.6, R63.2; no longer IC6.6, R54.2
- net N$21: now also IC7.2, R52.2, R60.1; no longer IC6.2, R42.1, R43.2
- net N$22: now also C19.1, IC7.1, R52.1, R61.2; no longer C20.1, IC6.1, R43.1, R47.2
- net N$23: now also C23.2, IC7.3, R46.2; no longer C19.2, IC6.3, R45.2
- net N$24: now also C19.2, R40.2, R46.1; no longer C20.2, R44.2, R45.1
- net N$25: now also C31.1, IC7.12, R75.2; no longer C21.1, IC6.12, R48.2
- net N$26: now also IC7.8, R71.2, R75.1; no longer IC6.8, R48.1, R50.2
- net N$27: now also IC7.9, R62.1, R71.1; no longer IC6.9, R49.1, R50.1
- net N$28: now also C28.2, IC7.7, R62.2; no longer C22.2, IC6.7, R49.2
- net N$29: now also C24.1, IC7.5, R47.2; no longer C23.1, IC6.5, R52.2
- net N$30: now also C28.1, R41.2, R47.1; no longer C22.1, R51.2, R52.1
- net N$31: now also IC7.10, R61.1, R70.2; no longer IC6.10, R46.2, R47.1
- net N$32: now also IC8.6, R55.1; no longer IC7.6, R66.1
- net N$33: now also IC8.2, R54.2, R64.1; no longer IC7.2, R55.1, R56.2
- net N$34: now also C20.1, IC8.1, R54.1, R65.2; no longer C25.1, IC7.1, R56.1, R60.2
- net N$35: now also C25.2, IC8.3, R48.2; no longer C24.2, IC7.3, R58.2
- net N$36: now also C20.2, R42.2, R48.1; no longer C25.2, R57.2, R58.1
- net N$37: now also C32.1, IC8.12, R76.2; no longer C26.1, IC7.12, R61.2
- net N$38: now also IC8.8, R73.2, R76.1; no longer IC7.8, R61.1, R63.2
- net N$39: now also IC8.9, R66.1, R73.1; no longer IC7.9, R62.1, R63.1
- net N$4: now also U2.1; no longer U1.1
- net N$40: now also C29.2, IC8.7, R55.2; no longer C27.2, IC7.7, R62.2
- net N$41: now also C26.1, IC8.5, R49.2; no longer C28.1, IC7.5, R65.2
- net N$42: now also C29.1, R43.2, R49.1; no longer C27.1, R64.2, R65.1
- net N$43: now also IC8.10, R65.1, R72.2; no longer IC7.10, R59.2, R60.1
- net N$45: now also R79.2; no longer R68.2
- net N$47: now also R80.2; no longer R69.2
- net N$48: now also R81.2; no longer R70.2
- net N$5: now also C18.1, IC6.1, R50.1, R57.2; no longer C15.1, IC5.1, R30.1, R34.2
- net N$50: now also C34.2, IC9.4; no longer C30.2, IC8.4
- net N$51: now also C34.1, IC9.2; no longer C30.1, IC8.2
- net N$52: now also C33.2, IC9.6; no longer C29.2, IC8.6
- net N$53: now also C33.1, IC9.5; no longer C29.1, IC8.5
- net N$54: now also C36.1, IC9.3; no longer C31.1, IC8.3
- net N$55: now also C37.1, IC9.7; no longer C32.1, IC8.7
- net N$56: now also C12.1, OK1.3, R7.2; no longer C43.1, OK4.3, R79.2
- net N$6: now also C21.2, IC6.3, R44.2; no longer C14.2, IC5.3, R32.2
- net N$65: now also LED3.C; no longer LED4.C
- net N$67: now also C38.2, R77.1, R78.1; no longer C34.2, R71.1, R72.1
- net N$69: now also Q1.1, R14.2; no longer Q4.1, R81.2
- net N$7: now also C18.2, R38.2, R44.1; no longer C15.2, R31.2, R32.1
- net N$70: now also C13.1, OK1.5, R8.2; no longer C44.1, OK4.5, R84.2
- net N$71: now also C14.1, OK1.7, R9.2; no longer C45.1, OK4.7, R89.2
- net N$72: now also C11.1, OK1.1, R6.2; no longer C42.1, OK4.1, R74.2
- net N$73: now also OK2.4, R16.2; no longer OK1.4, R12.2
- net N$74: now also OK2.1, R15.2; no longer OK1.1, R8.2
- net N$75: now also LED4.C; no longer LED5.C
- net N$76: now also LED5.A; no longer LED3.A
- net N$8: now also C30.1, IC6.12, R74.2; no longer C16.1, IC5.12, R35.2
- net N$9: now also IC6.8, R69.2, R74.1; no longer IC5.8, R35.1, R37.2
- net OSC1I: now also C45.2, IC10.39, Q2.2; no longer C38.2, IC9.39, Q1.2
- net OSC1O: now also C46.2, IC10.40, Q2.1; no longer C41.2, IC9.40, Q1.1
- net PGEC: now also IC10.44; no longer IC9.44
- net PGED: now also IC10.43; no longer IC9.43
- net RO1: now also IC10.61, R14.1; no longer IC9.61, R81.1
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Routing:
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Other:
- board text added: "+"
- board text added: "-"
- board text added: "SCX3 v1.1.0"
- board text removed: "+24V"
- board text removed: "GND"
- board text removed: "v1.0.0 rev.1"

Commit message: Release 1.2.0
Parts:
- removed C37, C38, C39, C40, C41: 100n, rcl:C0805
- removed IC9: MAX3221CAE, ServoController:SSOP16
- removed LED4: LED 3V3, led:SML1206
- removed LED7: LED STATE, led:SML1206
- removed R1: 2K2, rcl:R1206
- removed R4: 330, rcl:R0805
- removed R7: 1K, rcl:R0805
- removed RS232: RJ-9, SCX3:RJ-9
- added C47, C48, C49, C50: 100n, rcl:C0805
- added C55: 100n, rcl:UD-4X5,8_NICHICON
- added D2, D3: 1N4148, diode:D0805
- added D4: ESD5Z3.3, diode:SOD523
- added F2: 0.63A, fuse:TR5
- added IC13: MAX3089, MyLib:SO14
- added L2: 4,7uH, MyLib:DJNR6028
- added LED14: LED READY, led:SML1206
- added LED15: LED STATE, led:SML1206
- added LED16: LED ERROR, led:SML1206
- added LED19: TX, led:SML0603
- added LED20: RX, led:SML0603
- added Q3, Q4: BC848, transistor-npn:SOT23
- added R85, R88, R89: 100, rcl:R0805
- added R86, R87, R90: 4K7, rcl:R0805
- added R91: 10K, rcl:R0805
- added R92: 1K, rcl:R0805
- added R95, R96: 100, rcl:R0603
- added R97: 10K, rcl:R0603
- added RS485-IN, RS485-OUT: RJ-45-SH_RJSS-88-A22-E1V, MyLib:RJ-45M
- added S1: DIP-6_TDA06H0_SB1, MyLib:TDA06H0_S
- added USB: USB, MyLib:USB-B-PTH-VERTICAL
- C1: value 330uF -> 1nF/1KV; device rcl:E5-10,5 -> rcl:C1206
- C10: value 10uF -> 1uF
- C11, C14: value 100n -> 10uF
- C12: value 100n -> 1nF/1KV; device rcl:C0805 -> rcl:C1206
- C13: value 100n -> 10uF; device rcl:C0805 -> rcl:UD-4X5,8_NICHICON
- C15, C16, C17: value 10uF -> 100n
- C18: value 10n -> 100n
- C19, C20: value 10n -> 10uF
- C2: value 220uF -> 1uF; device rcl:E5-10,5 -> rcl:C0805
- C21: value 33n -> 10uF
- C23, C25, C30: value 33n -> 10n
- C27, C29: value 10n -> 33n
- C3: value 10uF -> 1000uF; device rcl:UD-4X5,8_NICHICON -> rcl:E5-10,5
- C33: value 100n -> 10n
- C34, C36: value 100n -> 33n
- C35: value 100n -> 10n; device rcl:UD-4X5,8_NICHICON -> rcl:C0805
- C43, C44: value 100n -> 27p
- C45, C46: value 27p -> 100n
- C5: value 1nF/1KV -> 10uF
- C6: value 1nF/1KV -> 1uF
- C7: value 10uF -> 1nF/1KV; device rcl:C0805 -> rcl:C1206
- C8: value 1uF -> 1nF/1KV; device rcl:C0805 -> rcl:C1206
- C9: value 1uF -> 330uF; device rcl:C0805 -> rcl:E5-10,5
- D1: value 1N4148SMD-0805 -> 1N4148
- ENCODER1, ENCODER2, ENCODER3, OUTPUT: device ServoController:F09VP -> con-subd:F09VP
- F1: value 3A -> 0.63A; device fuse:SH22,5 -> fuse:TR5
- IC1, OK2, OK3, OK4: device ServoController:DIL08 -> MyLib:DIL08
- IC10: value PIC32MK1024MCF064 -> M95040; device ServoController:QFN64-9X9 -> MyLib:SO8
- IC11: value M95040 -> PIC32MK1024MCF064; device SCX3:SO8 -> MyLib:QFN64-9X9
- IC6, IC7, IC8: device ServoController:DIL14 -> MyLib:DIL14
- ICSP: device ServoController:JP5 -> MyLib:JP5
- K1: device ServoController:G6K-2P-Y -> MyLib:G6K-2P-Y
- L1: device ServoController:DJNR6028 -> MyLib:DJNR6028
- LED1: value LED 24V -> (none); device led:SML1206 -> led:DUOLED-C-5MM
- LED2: value LED +12V -> (none); device led:SML1206 -> led:DUOLED-C-5MM
- LED3: value LED 5V -> LED +12V
- LED6: value LED READY -> LED 5V
- LED8: value LED ERROR -> LED 3V3
- OK1: device ServoController:DIL16 -> MyLib:DIL16
- R11, R13: value 4K7 -> 470; device rcl:R0805 -> rcl:R1206
- R15, R17: value 470 -> 1K
- R16, R18, R23, R24, R31: value 470 -> 4K7
- R19, R22: value 4K7 -> 1K
- R2, R9: value 1K -> 470; device rcl:R0805 -> rcl:R1206
- R25, R26, R29, R32, R34: value 4K7 -> 470
- R30: value 1K -> 470
- R38, R39, R40, R41, R42, R43: value 22K -> 4K7
- R44: value 10K -> 1K
- R45: value 10K -> 470
- R46: value 10K -> 47K
- R47, R48, R77: value 10K -> 22K
- R5: value 100 -> 1K
- R50, R54, R58, R76: value 22K -> 47K
- R56, R69: value 47K -> 10K
- R6: value 1K -> 330
- R60, R64, R68, R70, R73: value 47K -> 22K
- R62, R75: value 22K -> 10K
- R78: value 1K -> 22K
- R79, R81: value 100 -> 22K
- R8: value 1K -> 100
- R80: value 100 -> 47K
- R82: value 4K7 -> 10K
- R83: value 4K7 -> 22K
- R84: value 4K7 -> 47K
- U1: value AM6T-2412D-NZ -> AM6C-2412D-NZ; device SCX3:AM6T -> MyLib:AM6C
- U2: device ServoController:AM10CW-NZ -> MyLib:AM10CW-NZ
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Connections:
- net DO1H_CON renamed N$12
- removed net 24V: C1.+, C2.+, C4.1, C5.1, F1.2, INTERFACE.15, L1.A, LED1.A, U1.22, U1.23
- removed net N$12 (its old number): F1.1, POWER.1
- removed net N$3: LED1.C, R1.1
- removed net N$50: C34.2, IC9.4
- removed net N$51: C34.1, IC9.2
- removed net N$52: C33.2, IC9.6
- removed net N$53: C33.1, IC9.5
- removed net N$54: C36.1, IC9.3
- removed net N$55: C37.1, IC9.7
- removed net RS232_RX: IC9.8, RS232.2
- removed net RS232_TX: IC9.13, RS232.3
- new net 24V_1: C3.+, C4.1, D2.1, F1.2, L1.A
- new net 24V_2: C10.1, C9.+, D3.1, F2.2, L2.A
- new net 24V_SUPPLY: F1.1, F2.1, POWER.1, R2.1, R9.1
- new net H/!F: IC13.1, S1.12
- new net N$46: C1.1, L1.B, U1.1
- new net N$49: LED1.AR, Q3.3, R9.2
- new net N$57: Q3.1, R10.2
- new net N$59: LED1.AX, R11.1
- new net N$60: D2.2, R10.1, R11.2
- new net N$61: LED2.AR, Q4.3, R2.2
- new net N$66: Q4.1, R12.2
- new net N$68: LED2.AX, R13.1
- new net N$77: D3.2, R12.1, R13.2
- new net N$82: LED19.A, R95.2
- new net N$83: LED20.A, R96.2
- new net N$85: R97.1, S1.9
- new net RS485_A: IC13.12, RS485-IN.5, RS485-OUT.5
- new net RS485_B: IC13.11, RS485-IN.8, RS485-OUT.8
- new net RS485_Y: IC13.9, RS485-IN.1, RS485-OUT.1
- new net RS485_Z: IC13.10, RS485-IN.4, RS485-OUT.4
- new net RXP: IC13.13, S1.10
- new net SLR: IC13.6, R97.2, S1.8
- new net TXP: IC13.8, S1.11
- new net UART_!CTS: IC11.46, IC13.3, IC13.4
- new net UART_!RTR: IC11.45
- new net USB_D+: IC11.37, USB.D+
- new net USB_D-: IC11.36, USB.D-
- new net VBUS: IC11.34, USB.VBUS
- net !HOLD: now also IC10.7, R87.2; no longer IC11.7, R84.2
- net !MCLR: now also IC11.7, R92.2; no longer IC10.7, R78.2
- net !MSS: now also IC10.1, IC11.50, R86.2; no longer IC10.50, IC11.1, R83.2
- net !MWP: now also IC10.3, IC11.47, R90.2; no longer IC10.47, IC11.3, R82.2
- net +12V: now also C1.2, C2.1, C5.1, LED3.A, U1.3; no longer C5.2, C8.1, LED2.A, U1.14
- net -12V: now also C5.2, C6.2, C7.1, U1.5; no longer C6.1, C9.2, U1.11
- net 24VGND: now also C10.2, C12.2, C3.-, C7.2, C9.-, LED1.C, LED2.C, Q3.2, Q4.2; no longer C1.-, C2.-, C6.2, R1.2, U1.3
- net 3V3: now also C14.1, C46.2, C47.2, C48.1, C49.2, C50.1, C55.+, D4.C, IC10.8, IC11.10, IC11.19, IC11.26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; no longer C35.+, C39.2, C40.1, C41.2, C43.2, C44.1, C7.1, IC10.10, IC10.19, IC10.26, IC10.35, IC10.38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
- net 5V: now also C11.1, C13.+, C19.2, C20.2, C21.2, C8.2, LED6.A, R44.2; no longer C10.1, C15.2, C16.2, C17.2, C3.+, LED3.A, R30.2
- net CH1_A+: now also IC3.7; no longer IC3.5
- net CH1_A-: now also IC3.6; no longer IC3.4
- net CH1_B+: now also IC3.5; no longer IC3.7
- net CH1_B-: now also IC3.4, SJ5.2; no longer IC3.6, SJ3.2
- net CH1_DIR: now also IC11.21, R27.1; no longer IC10.21, R19.1
- net CH1_DIR_H: now also R29.1; no longer R16.1
- net CH1_H: now also IC11.2, R48.1; no longer IC10.2, R38.1
- net CH1_I-: now also SJ8.2; no longer SJ4.2
- net CH1_L: now also IC11.3, R55.1; no longer IC10.3, R39.1
- net CH1_QE_A: now also IC11.30, IC3.1, R38.1; no longer IC10.30, IC3.2, R27.1
- net CH1_QE_B: now also IC11.33, IC3.2, R35.1; no longer IC10.33, IC3.1, R28.1
- net CH1_QE_I: now also IC11.31, R41.1; no longer IC10.31, R29.1
- net CH1_STEP: now also IC11.18, R23.1; no longer IC10.18, R21.1
- net CH1_STEP_H: now also R25.1; no longer R15.1
- net CH2_A-: now also SJ3.2; no longer SJ5.2
- net CH2_DIR: now also IC11.32, OK3.6, R28.1; no longer IC10.32, OK4.6, R25.1
- net CH2_DIR_H: now also R30.1; no longer R24.1
- net CH2_DIR_L: now also OK3.3; no longer OK4.3
- net CH2_H: now also IC11.64, R61.1; no longer IC10.64, R40.1
- net CH2_I-: now also SJ9.2; no longer SJ7.2
- net CH2_L: now also IC11.1, R68.1; no longer IC10.1, R41.1
- net CH2_QE_A: now also IC11.23, R36.1; no longer IC10.23, R32.1
- net CH2_QE_B: now also IC11.22, R39.1; no longer IC10.22, R33.1
- net CH2_QE_I: now also IC11.16, R42.1; no longer IC10.16, R34.1
- net CH2_STEP: now also IC11.29, OK3.7, R24.1; no longer IC10.29, OK4.7, R26.1
- net CH2_STEP_H: now also R26.1; no longer R23.1
- net CH2_STEP_L: now also OK3.2; no longer OK4.2
- net CH3_A-: now also SJ4.2; no longer SJ8.2
- net CH3_B-: now also SJ7.2; no longer SJ9.2
- net CH3_DIR: now also IC11.24, OK4.6, R33.1; no longer IC10.24, OK3.6, R20.1
- net CH3_DIR_H: now also R34.1; no longer R18.1
- net CH3_DIR_L: now also OK4.3; no longer OK3.3
- net CH3_H: now also IC11.62, R74.1; no longer IC10.62, R42.1
- net CH3_L: now also IC11.63, R81.1; no longer IC10.63, R43.1
- net CH3_QE_A: now also IC11.13, R37.1; no longer IC10.13, R35.1
- net CH3_QE_B: now also IC11.14, R40.1; no longer IC10.14, R36.1
- net CH3_QE_I: now also IC11.17, R43.1; no longer IC10.17, R37.1
- net CH3_STEP: now also IC11.15, OK4.7, R31.1; no longer IC10.15, OK3.7, R22.1
- net CH3_STEP_H: now also R32.1; no longer R17.1
- net CH3_STEP_L: now also OK4.2; no longer OK3.2
- net DI1: now also IC11.4, R14.1; no longer IC10.4, R10.1
- net DI1_CON: now also R15.1; no longer R6.1
- net DI2: now also IC11.5, R16.1; no longer IC10.5, R11.1
- net DI2_CON: now also R17.1; no longer R7.1
- net DI3: now also IC11.6, R18.1; no longer IC10.6, R12.1
- net DI3_CON: now also R19.1; no longer R8.1
- net DI4: now also IC11.8, R21.1; no longer IC10.8, R13.1
- net DI4_CON: now also R22.1; no longer R9.1
- net DI_COM_CON: now also C15.2, C16.2, C17.2, C18.2; no longer C11.2, C12.2, C13.2, C14.2
- net DO1: now also IC11.52; no longer IC10.52
- net DO2: now also IC11.53; no longer IC10.53
- net DO3: now also IC11.11; no longer IC10.11
- net DO4: now also IC11.12; no longer IC10.12
- net GND: now also C11.2, C12.1, C13.-, C14.2, C19.1, C2.2, C20.1, C22.1, C27.1, C29.2, C32.1, C34.2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; no longer C10.2, C15.1, C16.1, C17.1, C22.2, C23.1, C25.1, C3.-, C30.2, C32.2, C35.-, C37.2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
- net LED_ERROR: now also IC11.60, R89.1; no longer IC10.60, R81.1
- net LED_READY: now also IC11.58, R85.1; no longer IC10.58, R79.1
- net LED_STATE: now also IC11.59, R88.1; no longer IC10.59, R80.1
- net MSCK: now also IC10.6, IC11.51; no longer IC10.51, IC11.6
- net MSDI: now also IC10.2, IC11.48; no longer IC10.48, IC11.2
- net MSDO: now also IC10.5, IC11.49; no longer IC10.49, IC11.5
- net N$1: now also R57.1, R58.2; no longer R51.1, R59.2
- net N$10: now also R53.1, R54.1; no longer R58.1, R69.1
- net N$11: now also C25.2, R53.2, R57.2; no longer C27.2, R51.2, R58.2
- net N$13: now also C26.1, R56.2; no longer C22.1, R45.2
- net N$14: now also C25.1, R55.2, R56.1; no longer C27.1, R39.2, R45.1
- net N$15: now also R50.2, R51.1; no longer R57.1, R68.2
- net N$16: now also OK3.4, R30.2; no longer OK4.4, R24.2
- net N$17: now also OK3.1, R26.2; no longer OK4.1, R23.2
- net N$18: now also OK4.4, R34.2; no longer OK3.4, R18.2
- net N$19: now also OK4.1, R32.2; no longer OK3.1, R17.2
- net N$2: now also R46.1, R47.2; no longer R50.2, R56.1
- net N$20: now also R70.1, R71.2; no longer R53.1, R63.2
- net N$21: now also R59.1, R60.2; no longer R52.2, R60.1
- net N$22: now also C28.1, R60.1, R64.2; no longer C19.1, R52.1, R61.2
- net N$23: now also C27.2, R62.2; no longer C23.2, R46.2
- net N$24: now also C28.2, R61.2, R62.1; no longer C19.2, R40.2, R46.1
- net N$25: now also C29.1, R65.2; no longer C31.1, R75.2
- net N$26: now also R65.1, R67.2; no longer R71.2, R75.1
- net N$27: now also R66.1, R67.1; no longer R62.1, R71.1
- net N$28: now also C30.2, R66.2, R70.2; no longer C28.2, R53.2, R62.2
- net N$29: now also C31.1, R69.2; no longer C24.1, R47.2
- net N$30: now also C30.1, R68.2, R69.1; no longer C28.1, R41.2, R47.1
- net N$31: now also R63.2, R64.1; no longer R61.1, R70.2
- net N$32: now also R83.1, R84.2; no longer R55.1, R67.2
- net N$33: now also R72.1, R73.2; no longer R54.2, R64.1
- net N$34: now also C33.1, R73.1, R77.2; no longer C20.1, R54.1, R65.2
- net N$35: now also C32.2, R75.2; no longer C25.2, R48.2
- net N$36: now also C33.2, R74.2, R75.1; no longer C20.2, R42.2, R48.1
- net N$37: now also C34.1, R78.2; no longer C32.1, R76.2
- net N$38: now also R78.1, R80.2; no longer R73.2, R76.1
- net N$39: now also R79.1, R80.1; no longer R66.1, R73.1
- net N$4: now also C8.1, L2.B; no longer L1.B
- net N$40: now also C35.2, R79.2, R83.2; no longer C29.2, R55.2, R66.2
- net N$41: now also C36.1, R82.2; no longer C26.1, R49.2
- net N$42: now also C35.1, R81.2, R82.1; no longer C29.1, R43.2, R49.1
- net N$43: now also R76.2, R77.1; no longer R65.1, R72.2
- net N$45: now also LED14.A, R85.2; no longer LED6.A, R79.2
- net N$47: now also LED15.A, R88.2; no longer LED7.A, R80.2
- net N$48: now also LED16.A, R89.2; no longer LED8.A, R81.2
- net N$5: now also C23.1, R47.1, R51.2; no longer C18.1, R50.1, R57.2
- net N$56: now also C16.1, R17.2; no longer C12.1, R7.2
- net N$58: now also LED3.C, R3.1; no longer LED2.C, R2.1
- net N$6: now also C22.2, R49.2; no longer C21.2, R44.2
- net N$65: now also LED6.C, R6.1; no longer LED3.C, R4.1
- net N$67: now also C45.2, R91.1, R92.1; no longer C38.2, R77.1, R78.1
- net N$69: now also R20.2; no longer R14.2
- net N$7: now also C23.2, R48.2, R49.1; no longer C18.2, R38.2, R44.1
- net N$70: now also C17.1, R19.2; no longer C13.1, R8.2
- net N$71: now also C18.1, R22.2; no longer C14.1, R9.2
- net N$72: now also C15.1, R15.2; no longer C11.1, R6.2
- net N$73: now also R29.2; no longer R16.2
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Routing:
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- added copper zone on layer 1, net N$3
- added copper zone on layer 16, net N$44
Other:
- board size 157 x 72 mm -> 170 x 73 mm
- board text added: "0.63A"
- board text added: "RX"
- board text added: "TX"
- board text added: "v1.2.0 rev.1"
- board text removed: "3A"
- board text removed: "SCX3 v1.1.0"

Commit message: [BROKEN] Rotated encoder 3 gate transoptor (IC5)
Only for the purpose of containing the concept of positioning the elements
Parts:
- removed C47, C48, C49, C50: 100n, rcl:C0805
- removed C55: 100n, rcl:UD-4X5,8_NICHICON
- removed D2, D3: 1N4148, diode:D0805
- removed D4: ESD5Z3.3, diode:SOD523
- removed F2: 0.63A, fuse:TR5
- removed IC13: MAX3089, MyLib:SO14
- removed L2: 4,7uH, MyLib:DJNR6028
- removed LED14: LED READY, led:SML1206
- removed LED15: LED STATE, led:SML1206
- removed LED16: LED ERROR, led:SML1206
- removed LED19: TX, led:SML0603
- removed LED20: RX, led:SML0603
- removed Q3, Q4: BC848, transistor-npn:SOT23
- removed R85, R88, R89: 100, rcl:R0805
- removed R86, R87, R90: 4K7, rcl:R0805
- removed R91: 10K, rcl:R0805
- removed R92: 1K, rcl:R0805
- removed R95, R96: 100, rcl:R0603
- removed R97: 10K, rcl:R0603
- removed RS485-IN, RS485-OUT: RJ-45-SH_RJSS-88-A22-E1V, MyLib:RJ-45M
- removed S1: DIP-6_TDA06H0_SB1, MyLib:TDA06H0_S
- removed USB: USB, MyLib:USB-B-PTH-VERTICAL
- added C37, C38, C39, C40, C41: 100n, rcl:C0805
- added IC9: MAX3221CAE, ServoController:SSOP16
- added LED4: LED 3V3, led:SML1206
- added LED7: LED STATE, led:SML1206
- added R1: 2K2, rcl:R1206
- added R4: 330, rcl:R0805
- added R7: 1K, rcl:R0805
- added RS232: RJ-9, SCX3:RJ-9
- C1: value 1nF/1KV -> 330uF; device rcl:C1206 -> rcl:E5-10,5
- C10: value 1uF -> 10uF
- C11, C14: value 10uF -> 100n
- C12: value 1nF/1KV -> 100n; device rcl:C1206 -> rcl:C0805
- C13: value 10uF -> 100n; device rcl:UD-4X5,8_NICHICON -> rcl:C0805
- C15, C16, C17: value 100n -> 10uF
- C18: value 100n -> 10n
- C19, C20: value 10uF -> 10n
- C2: value 1uF -> 220uF; device rcl:C0805 -> rcl:E5-10,5
- C21: value 10uF -> 33n
- C23, C25, C30: value 10n -> 33n
- C27, C29: value 33n -> 10n
- C3: value 1000uF -> 10uF; device rcl:E5-10,5 -> rcl:UD-4X5,8_NICHICON
- C33: value 10n -> 100n
- C34, C36: value 33n -> 100n
- C35: value 10n -> 100n; device rcl:C0805 -> rcl:UD-4X5,8_NICHICON
- C43, C44: value 27p -> 100n
- C45, C46: value 100n -> 27p
- C5: value 10uF -> 1nF/1KV
- C6: value 1uF -> 1nF/1KV
- C7: value 1nF/1KV -> 10uF; device rcl:C1206 -> rcl:C0805
- C8: value 1nF/1KV -> 1uF; device rcl:C1206 -> rcl:C0805
- C9: value 330uF -> 1uF; device rcl:E5-10,5 -> rcl:C0805
- D1: value 1N4148 -> 1N4148SMD-0805
- ENCODER1, ENCODER2, ENCODER3, OUTPUT: device con-subd:F09VP -> ServoController:F09VP
- F1: value 0.63A -> 3A; device fuse:TR5 -> fuse:SH22,5
- IC1, OK2, OK3, OK4: device MyLib:DIL08 -> ServoController:DIL08
- IC10: value M95040 -> PIC32MK1024MCF064; device MyLib:SO8 -> ServoController:QFN64-9X9
- IC11: value PIC32MK1024MCF064 -> M95040; device MyLib:QFN64-9X9 -> SCX3:SO8
- IC6, IC7, IC8: device MyLib:DIL14 -> ServoController:DIL14
- ICSP: device MyLib:JP5 -> ServoController:JP5
- K1: device MyLib:G6K-2P-Y -> ServoController:G6K-2P-Y
- L1: device MyLib:DJNR6028 -> ServoController:DJNR6028
- LED1: value (none) -> LED 24V; device led:DUOLED-C-5MM -> led:SML1206
- LED2: value (none) -> LED +12V; device led:DUOLED-C-5MM -> led:SML1206
- LED3: value LED +12V -> LED 5V
- LED6: value LED 5V -> LED READY
- LED8: value LED 3V3 -> LED ERROR
- OK1: device MyLib:DIL16 -> ServoController:DIL16
- R11, R13: value 470 -> 4K7; device rcl:R1206 -> rcl:R0805
- R15, R17: value 1K -> 470
- R16, R18, R23, R24, R31: value 4K7 -> 470
- R19, R22: value 1K -> 4K7
- R2, R9: value 470 -> 1K; device rcl:R1206 -> rcl:R0805
- R25, R26, R29, R32, R34: value 470 -> 4K7
- R30: value 470 -> 1K
- R38, R39, R40, R41, R42, R43: value 4K7 -> 22K
- R44: value 1K -> 10K
- R45: value 470 -> 10K
- R46: value 47K -> 10K
- R47, R48, R77: value 22K -> 10K
- R5: value 1K -> 100
- R50, R54, R58, R76: value 47K -> 22K
- R56, R69: value 10K -> 47K
- R6: value 330 -> 1K
- R60, R64, R68, R70, R73: value 22K -> 47K
- R62, R75: value 10K -> 22K
- R78: value 22K -> 1K
- R79, R81: value 22K -> 100
- R8: value 100 -> 1K
- R80: value 47K -> 100
- R82: value 10K -> 4K7
- R83: value 22K -> 4K7
- R84: value 47K -> 4K7
- U1: value AM6C-2412D-NZ -> AM6T-2412D-NZ; device MyLib:AM6C -> SCX3:AM6T
- U2: device MyLib:AM10CW-NZ -> ServoController:AM10CW-NZ
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Connections:
- net N$12 renamed DO1H_CON
- removed net 24V_1: C3.+, C4.1, D2.1, F1.2, L1.A
- removed net 24V_2: C10.1, C9.+, D3.1, F2.2, L2.A
- removed net 24V_SUPPLY: F1.1, F2.1, POWER.1, R2.1, R9.1
- removed net H/!F: IC13.1, S1.12
- removed net N$46: C1.1, L1.B, U1.1
- removed net N$49: LED1.AR, Q3.3, R9.2
- removed net N$57: Q3.1, R10.2
- removed net N$59: LED1.AX, R11.1
- removed net N$60: D2.2, R10.1, R11.2
- removed net N$61: LED2.AR, Q4.3, R2.2
- removed net N$66: Q4.1, R12.2
- removed net N$68: LED2.AX, R13.1
- removed net N$77: D3.2, R12.1, R13.2
- removed net N$82: LED19.A, R95.2
- removed net N$83: LED20.A, R96.2
- removed net N$85: R97.1, S1.9
- removed net RS485_A: IC13.12, RS485-IN.5, RS485-OUT.5
- removed net RS485_B: IC13.11, RS485-IN.8, RS485-OUT.8
- removed net RS485_Y: IC13.9, RS485-IN.1, RS485-OUT.1
- removed net RS485_Z: IC13.10, RS485-IN.4, RS485-OUT.4
- removed net RXP: IC13.13, S1.10
- removed net SLR: IC13.6, R97.2, S1.8
- removed net TXP: IC13.8, S1.11
- removed net UART_!CTS: IC11.46, IC13.3, IC13.4
- removed net UART_!RTR: IC11.45
- removed net USB_D+: IC11.37, USB.D+
- removed net USB_D-: IC11.36, USB.D-
- removed net VBUS: IC11.34, USB.VBUS
- new net 24V: C1.+, C2.+, C4.1, C5.1, F1.2, INTERFACE.15, L1.A, LED1.A, U1.22, U1.23
- new net N$12: F1.1, POWER.1
- new net N$3: LED1.C, R1.1
- new net N$50: C34.2, IC9.4
- new net N$51: C34.1, IC9.2
- new net N$52: C33.2, IC9.6
- new net N$53: C33.1, IC9.5
- new net N$54: C36.1, IC9.3
- new net N$55: C37.1, IC9.7
- new net RS232_RX: IC9.8, RS232.2
- new net RS232_TX: IC9.13, RS232.3
- net !HOLD: now also IC11.7, R84.2; no longer IC10.7, R87.2
- net !MCLR: now also IC10.7, R78.2; no longer IC11.7, R92.2
- net !MSS: now also IC10.50, IC11.1, R83.2; no longer IC10.1, IC11.50, R86.2
- net !MWP: now also IC10.47, IC11.3, R82.2; no longer IC10.3, IC11.47, R90.2
- net +12V: now also C5.2, C8.1, LED2.A, U1.14; no longer C1.2, C2.1, C5.1, LED3.A, U1.3
- net -12V: now also C6.1, C9.2, U1.11; no longer C5.2, C6.2, C7.1, U1.5
- net 24VGND: now also C1.-, C2.-, C6.2, R1.2, U1.3; no longer C10.2, C12.2, C3.-, C7.2, C9.-, LED1.C, LED2.C, Q3.2, Q4.2
- net 3V3: now also C35.+, C39.2, C40.1, C41.2, C43.2, C44.1, C7.1, IC10.10, IC10.19, IC10.26, IC10.35, IC10.38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; no longer C14.1, C46.2, C47.2, C48.1, C49.2, C50.1, C55.+, D4.C, IC10.8, IC11.10, IC11.19, IC11.26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
- net 5V: now also C10.1, C15.2, C16.2, C17.2, C3.+, LED3.A, R30.2; no longer C11.1, C13.+, C19.2, C20.2, C21.2, C8.2, LED6.A, R44.2
- net CH1_A+: now also IC3.5; no longer IC3.7
- net CH1_A-: now also IC3.4; no longer IC3.6
- net CH1_B+: now also IC3.7; no longer IC3.5
- net CH1_B-: now also IC3.6, SJ3.2; no longer IC3.4, SJ5.2
- net CH1_DIR: now also IC10.21, R19.1; no longer IC11.21, R27.1
- net CH1_DIR_H: now also R16.1; no longer R29.1
- net CH1_H: now also IC10.2, R38.1; no longer IC11.2, R48.1
- net CH1_I-: now also SJ4.2; no longer SJ8.2
- net CH1_L: now also IC10.3, R39.1; no longer IC11.3, R55.1
- net CH1_QE_A: now also IC10.30, IC3.2, R27.1; no longer IC11.30, IC3.1, R38.1
- net CH1_QE_B: now also IC10.33, IC3.1, R28.1; no longer IC11.33, IC3.2, R35.1
- net CH1_QE_I: now also IC10.31, R29.1; no longer IC11.31, R41.1
- net CH1_STEP: now also IC10.18, R21.1; no longer IC11.18, R23.1
- net CH1_STEP_H: now also R15.1; no longer R25.1
- net CH2_A-: now also SJ5.2; no longer SJ3.2
- net CH2_DIR: now also IC10.32, OK4.6, R25.1; no longer IC11.32, OK3.6, R28.1
- net CH2_DIR_H: now also R24.1; no longer R30.1
- net CH2_DIR_L: now also OK4.3; no longer OK3.3
- net CH2_H: now also IC10.64, R40.1; no longer IC11.64, R61.1
- net CH2_I-: now also SJ7.2; no longer SJ9.2
- net CH2_L: now also IC10.1, R41.1; no longer IC11.1, R68.1
- net CH2_QE_A: now also IC10.23, R32.1; no longer IC11.23, R36.1
- net CH2_QE_B: now also IC10.22, R33.1; no longer IC11.22, R39.1
- net CH2_QE_I: now also IC10.16, R34.1; no longer IC11.16, R42.1
- net CH2_STEP: now also IC10.29, OK4.7, R26.1; no longer IC11.29, OK3.7, R24.1
- net CH2_STEP_H: now also R23.1; no longer R26.1
- net CH2_STEP_L: now also OK4.2; no longer OK3.2
- net CH3_A-: now also SJ8.2; no longer SJ4.2
- net CH3_B-: now also SJ9.2; no longer SJ7.2
- net CH3_DIR: now also IC10.24, OK3.6, R20.1; no longer IC11.24, OK4.6, R33.1
- net CH3_DIR_H: now also R18.1; no longer R34.1
- net CH3_DIR_L: now also OK3.3; no longer OK4.3
- net CH3_H: now also IC10.62, R42.1; no longer IC11.62, R74.1
- net CH3_L: now also IC10.63, R43.1; no longer IC11.63, R81.1
- net CH3_QE_A: now also IC10.13, R35.1; no longer IC11.13, R37.1
- net CH3_QE_B: now also IC10.14, R36.1; no longer IC11.14, R40.1
- net CH3_QE_I: now also IC10.17, R37.1; no longer IC11.17, R43.1
- net CH3_STEP: now also IC10.15, OK3.7, R22.1; no longer IC11.15, OK4.7, R31.1
- net CH3_STEP_H: now also R17.1; no longer R32.1
- net CH3_STEP_L: now also OK3.2; no longer OK4.2
- net DI1: now also IC10.4, R10.1; no longer IC11.4, R14.1
- net DI1_CON: now also R6.1; no longer R15.1
- net DI2: now also IC10.5, R11.1; no longer IC11.5, R16.1
- net DI2_CON: now also R7.1; no longer R17.1
- net DI3: now also IC10.6, R12.1; no longer IC11.6, R18.1
- net DI3_CON: now also R8.1; no longer R19.1
- net DI4: now also IC10.8, R13.1; no longer IC11.8, R21.1
- net DI4_CON: now also R9.1; no longer R22.1
- net DI_COM_CON: now also C11.2, C12.2, C13.2, C14.2; no longer C15.2, C16.2, C17.2, C18.2
- net DO1: now also IC10.52; no longer IC11.52
- net DO2: now also IC10.53; no longer IC11.53
- net DO3: now also IC10.11; no longer IC11.11
- net DO4: now also IC10.12; no longer IC11.12
- net GND: now also C10.2, C15.1, C16.1, C17.1, C22.2, C23.1, C25.1, C3.-, C30.2, C32.2, C35.-, C37.2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; no longer C11.2, C12.1, C13.-, C14.2, C19.1, C2.2, C20.1, C22.1, C27.1, C29.2, C32.1, C34.2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
- net LED_ERROR: now also IC10.60, R81.1; no longer IC11.60, R89.1
- net LED_READY: now also IC10.58, R79.1; no longer IC11.58, R85.1
- net LED_STATE: now also IC10.59, R80.1; no longer IC11.59, R88.1
- net MSCK: now also IC10.51, IC11.6; no longer IC10.6, IC11.51
- net MSDI: now also IC10.48, IC11.2; no longer IC10.2, IC11.48
- net MSDO: now also IC10.49, IC11.5; no longer IC10.5, IC11.49
- net N$1: now also R51.1, R59.2; no longer R57.1, R58.2
- net N$10: now also R58.1, R69.1; no longer R53.1, R54.1
- net N$11: now also C27.2, R51.2, R58.2; no longer C25.2, R53.2, R57.2
- net N$13: now also C22.1, R45.2; no longer C26.1, R56.2
- net N$14: now also C27.1, R39.2, R45.1; no longer C25.1, R55.2, R56.1
- net N$15: now also R57.1, R68.2; no longer R50.2, R51.1
- net N$16: now also OK4.4, R24.2; no longer OK3.4, R30.2
- net N$17: now also OK4.1, R23.2; no longer OK3.1, R26.2
- net N$18: now also OK3.4, R18.2; no longer OK4.4, R34.2
- net N$19: now also OK3.1, R17.2; no longer OK4.1, R32.2
- net N$2: now also R50.2, R56.1; no longer R46.1, R47.2
- net N$20: now also R53.1, R63.2; no longer R70.1, R71.2
- net N$21: now also R52.2, R60.1; no longer R59.1, R60.2
- net N$22: now also C19.1, R52.1, R61.2; no longer C28.1, R60.1, R64.2
- net N$23: now also C23.2, R46.2; no longer C27.2, R62.2
- net N$24: now also C19.2, R40.2, R46.1; no longer C28.2, R61.2, R62.1
- net N$25: now also C31.1, R75.2; no longer C29.1, R65.2
- net N$26: now also R71.2, R75.1; no longer R65.1, R67.2
- net N$27: now also R62.1, R71.1; no longer R66.1, R67.1
- net N$28: now also C28.2, R53.2, R62.2; no longer C30.2, R66.2, R70.2
- net N$29: now also C24.1, R47.2; no longer C31.1, R69.2
- net N$30: now also C28.1, R41.2, R47.1; no longer C30.1, R68.2, R69.1
- net N$31: now also R61.1, R70.2; no longer R63.2, R64.1
- net N$32: now also R55.1, R67.2; no longer R83.1, R84.2
- net N$33: now also R54.2, R64.1; no longer R72.1, R73.2
- net N$34: now also C20.1, R54.1, R65.2; no longer C33.1, R73.1, R77.2
- net N$35: now also C25.2, R48.2; no longer C32.2, R75.2
- net N$36: now also C20.2, R42.2, R48.1; no longer C33.2, R74.2, R75.1
- net N$37: now also C32.1, R76.2; no longer C34.1, R78.2
- net N$38: now also R73.2, R76.1; no longer R78.1, R80.2
- net N$39: now also R66.1, R73.1; no longer R79.1, R80.1
- net N$4: now also L1.B; no longer C8.1, L2.B
- net N$40: now also C29.2, R55.2, R66.2; no longer C35.2, R79.2, R83.2
- net N$41: now also C26.1, R49.2; no longer C36.1, R82.2
- net N$42: now also C29.1, R43.2, R49.1; no longer C35.1, R81.2, R82.1
- net N$43: now also R65.1, R72.2; no longer R76.2, R77.1
- net N$45: now also LED6.A, R79.2; no longer LED14.A, R85.2
- net N$47: now also LED7.A, R80.2; no longer LED15.A, R88.2
- net N$48: now also LED8.A, R81.2; no longer LED16.A, R89.2
- net N$5: now also C18.1, R50.1, R57.2; no longer C23.1, R47.1, R51.2
- net N$56: now also C12.1, R7.2; no longer C16.1, R17.2
- net N$58: now also LED2.C, R2.1; no longer LED3.C, R3.1
- net N$6: now also C21.2, R44.2; no longer C22.2, R49.2
- net N$65: now also LED3.C, R4.1; no longer LED6.C, R6.1
- net N$67: now also C38.2, R77.1, R78.1; no longer C45.2, R91.1, R92.1
- net N$69: now also R14.2; no longer R20.2
- net N$7: now also C18.2, R38.2, R44.1; no longer C23.2, R48.2, R49.1
- net N$70: now also C13.1, R8.2; no longer C17.1, R19.2
- net N$71: now also C14.1, R9.2; no longer C18.1, R22.2
- net N$72: now also C11.1, R6.2; no longer C15.1, R15.2
- net N$73: now also R16.2; no longer R29.2
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Routing:
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- removed copper zone on layer 1, net N$3
- removed copper zone on layer 16, net N$44
Other:
- board size 170 x 73 mm -> 159 x 73 mm
- board text added: "3A"
- board text removed: "0.63A"
- board text removed: "RX"
- board text removed: "TX"
